Commit message: Update robot model to version 4

File: catkin_ws/src/car_robot_model/urdf/include/platform.xacro (robot description, xacro)
@@ -5,4 +5,6 @@
   <xacro:property name="wheel_width" value="0.001" />
   <link name="base_link">
+  </link>
+  <link name="body">
     <inertial>
       <mass value="6" />
@@ -17,5 +19,5 @@
         <mesh filename="package://car_robot_model/meshes/chassis.stl"/>
       </geometry>
-      <material name="Grey" />
+      <material name="Black" />
     </visual>
     <collision>
@@ -26,6 +28,11 @@
     </collision>
   </link>
+  <joint name="base_link_to_body" type="fixed">
+    <origin xyz="0.0 0 0.005" rpy="0 0 0" />
+    <parent link="base_link" />
+    <child link="body" />
+  </joint>
   <joint name="base_link_rear_left_wheel_joint" type="revolute">
-    <origin xyz="0.0 -0.0825 0" rpy="${PI/2.0} 0 0" />
+    <origin xyz="0.0 -0.0825 0.03" rpy="${PI/2.0} 0 0" />
     <axis xyz="0 0 1" />
     <anchor xyz="0 0 0" />
@@ -37,8 +44,8 @@
     <type>transmission_interface/SimpleTransmission</type>
     <joint name="base_link_rear_left_wheel_joint">
-      <hardwareInterface>EffortJointInterface</hardwareInterface>
+      <hardwareInterface>hardware_interface/EffortJointInterface</hardwareInterface>
     </joint>
     <actuator name="rear_left_motor">
-      <hardwareInterface>EffortJointInterface</hardwareInterface>
+      <hardwareInterface>hardware_interface/EffortJointInterface</hardwareInterface>
       <mechanicalReduction>1</mechanicalReduction>
     </actuator>
@@ -67,5 +74,5 @@
   </link>
   <joint name="base_link_rear_right_wheel_joint" type="revolute">
-    <origin xyz="0.0 0.0825 0" rpy="-${PI/2.0} 0 0" />
+    <origin xyz="0.0 0.0825 0.03" rpy="-${PI/2.0} 0 0" />
     <axis xyz="0 0 1" />
     <anchor xyz="0 0 0" />
@@ -77,8 +84,8 @@
     <type>transmission_interface/SimpleTransmission</type>
     <joint name="base_link_rear_right_wheel_joint">
-      <hardwareInterface>EffortJointInterface</hardwareInterface>
+      <hardwareInterface>hardware_interface/EffortJointInterface</hardwareInterface>
     </joint>
     <actuator name="rear_right_motor">
-      <hardwareInterface>EffortJointInterface</hardwareInterface>
+      <hardwareInterface>hardware_interface/EffortJointInterface</hardwareInterface>
       <mechanicalReduction>1</mechanicalReduction>
     </actuator>
@@ -107,5 +114,5 @@
   </link>
   <joint name="base_link_front_left_axel_joint" type="revolute">
-    <origin xyz="0.260 -0.0825 0" rpy="${PI/2.0} 0 0" />
+    <origin xyz="0.260 -0.0825 0.03" rpy="${PI/2.0} 0 0" />
     <axis xyz="0 1 0" />
     <anchor xyz="0 0 0" />
@@ -118,8 +125,8 @@
     <type>transmission_interface/SimpleTransmission</type>
     <joint name="base_link_front_left_axel_joint">
-      <hardwareInterface>EffortJointInterface</hardwareInterface>
+      <hardwareInterface>hardware_interface/EffortJointInterface</hardwareInterface>
     </joint>
     <actuator name="front_left_axel_motor">
-      <hardwareInterface>EffortJointInterface</hardwareInterface>
+      <hardwareInterface>hardware_interface/EffortJointInterface</hardwareInterface>
       <mechanicalReduction>1</mechanicalReduction>
     </actuator>
@@ -145,8 +152,8 @@
     <type>transmission_interface/SimpleTransmission</type>
     <joint name="front_left_axel_front_left_wheel_joint">
-      <hardwareInterface>EffortJointInterface</hardwareInterface>
+      <hardwareInterface>hardware_interface/EffortJointInterface</hardwareInterface>
     </joint>
     <actuator name="front_left_wheel_motor">
-      <hardwareInterface>EffortJointInterface</hardwareInterface>
+      <hardwareInterface>hardware_interface/EffortJointInterface</hardwareInterface>
       <mechanicalReduction>1</mechanicalReduction>
     </actuator>
@@ -175,5 +182,5 @@
   </link>
   <joint name="base_link_front_right_axel_joint" type="revolute">
-    <origin xyz="0.260 0.0825 0" rpy="-${PI/2.0} 0 0" />
+    <origin xyz="0.260 0.0825 0.03" rpy="-${PI/2.0} 0 0" />
     <axis xyz="0 1 0" />
     <anchor xyz="0 0 0" />
@@ -186,8 +193,8 @@
     <type>transmission_interface/SimpleTransmission</type>
     <joint name="base_link_front_right_axel_joint">
-      <hardwareInterface>EffortJointInterface</hardwareInterface>
+      <hardwareInterface>hardware_interface/EffortJointInterface</hardwareInterface>
     </joint>
     <actuator name="front_right_axel_motor">
-      <hardwareInterface>EffortJointInterface</hardwareInterface>
+      <hardwareInterface>hardware_interface/EffortJointInterface</hardwareInterface>
       <mechanicalReduction>1</mechanicalReduction>
     </actuator>
@@ -213,8 +220,8 @@
     <type>transmission_interface/SimpleTransmission</type>
     <joint name="front_right_axel_front_right_wheel_joint">
-      <hardwareInterface>EffortJointInterface</hardwareInterface>
+      <hardwareInterface>hardware_interface/EffortJointInterface</hardwareInterface>
     </joint>
     <actuator name="front_right_wheel_motor">
-      <hardwareInterface>EffortJointInterface</hardwareInterface>
+      <hardwareInterface>hardware_interface/EffortJointInterface</hardwareInterface>
       <mechanicalReduction>1</mechanicalReduction>
     </actuator>

File: catkin_ws/src/car_robot_model/urdf/include/sensors.xacro (robot description, xacro)
@@ -28,5 +28,5 @@
     <parent link="base_link"/>
     <child link="sensor_board"/>
-    <origin xyz="0 0 0.0415" rpy="0 0 0"/>
+    <origin xyz="0 0 0.07" rpy="0 0 0"/>
   </joint>
   <link name="camera_board">
@@ -86,5 +86,27 @@
     <parent link="sensor_board"/>
     <child link="imu"/>
-    <origin xyz="0.239 0.02 0.0025" rpy="0 0 ${PI/2}"/>
+    <origin xyz="0.035 -0.035 0.0025" rpy="0 0 ${PI/2}"/>
+  </joint>
+  <!-- Odroid -->
+  <link name="odroid">
+    <inertial>
+      <mass value="0.2000000" />
+      <origin xyz="0.00000000 0.00000000 0.00000000" rpy="0 0 0"/>
+      <inertia ixx="0.00000000" ixy="0.0" ixz="0.0"
+               iyy="0.00000000" iyz="0.0"
+               izz="0.00000000" />
+    </inertial>
+    <visual>
+      <origin xyz="0 0 0.01" rpy="0 0 0" />
+      <geometry>
+        <box size="0.06 0.08 0.015" />
+      </geometry>
+      <material name="Black" />
+    </visual>
+  </link>
+  <joint name="joint_sensor_board_to_odroid" type="fixed" >
+    <parent link="sensor_board"/>
+    <child link="odroid"/>
+    <origin xyz="-0.04 0 0" rpy="0 0 0"/>
   </joint>
   <!-- RP_LIDAR -->
@@ -114,9 +136,9 @@
     <parent link="sensor_board"/>
     <child link="laser"/>
-    <origin xyz="0.10445 0 0.0333" rpy="0 0 -${PI}"/>
+    <origin xyz="0.25 0 0.0333" rpy="0 0 0"/>
   </joint>
   <!-- top camera -->
-  <xacro:property name="top_camera_name" value="top_camera" />
-  <link name="${top_camera_name}">
+  <!--  <xacro:property name="top_camera_name" value="top_camera" />-->
+  <link name="top_camera">
     <inertial>
       <mass value="0.1600000" />
@@ -140,14 +162,14 @@
     </collision>
   </link>
-  <joint name="joint_camera_board_to_${top_camera_name}" type="fixed" >
+  <joint name="joint_camera_board_to_top_camera" type="fixed" >
     <parent link="camera_board"/>
-    <child link="${top_camera_name}"/>
+    <child link="top_camera"/>
     <origin xyz="0.019 0 0.0405" rpy="0 -${PI/2} ${PI}"/>
   </joint>
-  <link name="${top_camera_name}_optical">
-  </link>
-  <joint name="joint_${top_camera_name}_to_${top_camera_name}_optical" type="fixed" >
-    <parent link="${top_camera_name}"/>
-    <child link="${top_camera_name}_optical"/>
+  <link name="top_camera_optical">
+  </link>
+  <joint name="joint_top_camera_to_top_camera_optical" type="fixed" >
+    <parent link="top_camera"/>
+    <child link="top_camera_optical"/>
     <origin xyz="0.0 0 0.0" rpy="-${PI/2} 0 -${PI/2}"/>
   </joint>
