Commit message: Use camera_joint for calibration

File: catkin_ws/src/car_robot_model/urdf/include/_d435.urdf.xacro (robot description, xacro)
@@ -27,5 +27,5 @@
     <xacro:property name="d435_cam_depth_pz" value="${d435_cam_height/2}"/>
     <material name="aluminum">
-	  <color rgba="0.5 0.5 0.5 1"/>
+      <color rgba="0.5 0.5 0.5 1"/>
     </material>
     <!-- camera body, with origin at bottom screw mount -->
@@ -33,12 +33,18 @@
       <xacro:insert_block name="origin" />
       <parent link="${parent}"/>
+      <child link="camera_bottom_screw_frame" />
+    </joint>
+    <link name="camera_bottom_screw_frame"/>
+    <joint name="camera_link_joint" type="fixed">
+      <origin xyz="0 ${d435_cam_depth_py} ${d435_cam_depth_pz}" rpy="0 0 0"/>
+      <parent link="camera_bottom_screw_frame"/>
       <child link="camera_link" />
     </joint>
     <link name="camera_link">
       <visual>
-      <origin xyz="${d435_cam_mount_from_center_offset} 0.0 ${d435_cam_height/2}" rpy="${M_PI/2} 0 ${M_PI/2}"/>
+        <origin xyz="${d435_cam_mount_from_center_offset} ${-d435_cam_depth_py} 0" rpy="${M_PI/2} 0 ${M_PI/2}"/>
         <geometry>
           <!-- <box size="${d435_cam_width} ${d435_cam_height} ${d435_cam_depth}"/> -->
-	  <mesh filename="package://car_robot_model/meshes/d435.dae" />
+          <mesh filename="package://realsense2_camera/meshes/d435.dae" />
           <!--<mesh filename="package://realsense2_camera/meshes/d435/d435.dae" />-->
         </geometry>
@@ -46,7 +52,7 @@
       </visual>
       <collision>
-        <origin xyz="0.0 0.0 ${d435_cam_height/2}" rpy="0 0 0"/>
+        <origin xyz="0 ${-d435_cam_depth_py} 0" rpy="0 0 0"/>
         <geometry>
-        <box size="${d435_cam_depth} ${d435_cam_width} ${d435_cam_height}"/>
+          <box size="${d435_cam_depth} ${d435_cam_width} ${d435_cam_height}"/>
         </geometry>
       </collision>
@@ -60,5 +66,5 @@
     <!-- camera depth joints and links -->
     <joint name="camera_depth_joint" type="fixed">
-      <origin xyz="${d435_cam_depth_px} ${d435_cam_depth_py} ${d435_cam_depth_pz}" rpy="0 0 0"/>
+      <origin xyz="0 0 0" rpy="0 0 0"/>
       <parent link="camera_link"/>
       <child link="camera_depth_frame" />

Commit message: Remove upper aruco marker and use it as calibration marker

File: catkin_ws/src/car_robot_model/urdf/include/_d435.urdf.xacro (robot description, xacro)
@@ -46,5 +46,5 @@
         <geometry>
           <!-- <box size="${d435_cam_width} ${d435_cam_height} ${d435_cam_depth}"/> -->
-          <mesh filename="package://realsense2_camera/meshes/d435.dae" />
+          <mesh filename="package://car_robot_model/meshes/d435.dae" />
           <!--<mesh filename="package://realsense2_camera/meshes/d435/d435.dae" />-->
         </geometry>

File: catkin_ws/src/car_robot_model/urdf/include/sensors.xacro (robot description, xacro)
@@ -114,86 +114,9 @@
     <!-- Aruco Marker -->
     <link name="marker">
-        <inertial>
-            <mass value="0.2000000"/>
-            <origin xyz="0.00000000 0.00000000 0.00000000" rpy="0 0 0"/>
-            <inertia ixx="0.00000000" ixy="0.0" ixz="0.0"
-                     iyy="0.00000000" iyz="0.0"
-                     izz="0.00000000"/>
-        </inertial>
-        <visual>
-            <origin xyz="0 0 0.003" rpy="0 0 0"/>
-            <geometry>
-                <box size="0.12 0.12 0.002"/>
-            </geometry>
-            <material name="White"/>
-        </visual>
-        <visual>
-            <origin xyz="0.0 0.0 0.004" rpy="0 0 0"/>
-            <geometry>
-                <box size="0.09 0.09 0.002"/>
-            </geometry>
-            <material name="Black"/>
-        </visual>
-        <visual>
-            <origin xyz="0.0225 0.0225 0.005" rpy="0 0 0"/>
-            <geometry>
-                <box size="0.015 0.015 0.002"/>
-            </geometry>
-            <material name="White"/>
-        </visual>
-        <visual>
-            <origin xyz="0.0225 0.0075 0.005" rpy="0 0 0"/>
-            <geometry>
-                <box size="0.015 0.015 0.002"/>
-            </geometry>
-            <material name="White"/>
-        </visual>
-        <visual>
-            <origin xyz="0.0225 -0.0075 0.005" rpy="0 0 0"/>
-            <geometry>
-                <box size="0.015 0.015 0.002"/>
-            </geometry>
-            <material name="White"/>
-        </visual>
-        <visual>
-            <origin xyz="0.0075 0.0225 0.005" rpy="0 0 0"/>
-            <geometry>
-                <box size="0.015 0.015 0.002"/>
-            </geometry>
-            <material name="White"/>
-        </visual>
-        <visual>
-            <origin xyz="0.0075 -0.0075 0.005" rpy="0 0 0"/>
-            <geometry>
-                <box size="0.015 0.015 0.002"/>
-            </geometry>
-            <material name="White"/>
-        </visual>
-        <visual>
-            <origin xyz="0.0075 -0.0225 0.005" rpy="0 0 0"/>
-            <geometry>
-                <box size="0.015 0.015 0.002"/>
-            </geometry>
-            <material name="White"/>
-        </visual>
-        <visual>
-            <origin xyz="-0.0075 0.0075 0.005" rpy="0 0 0"/>
-            <geometry>
-                <box size="0.015 0.015 0.002"/>
-            </geometry>
-            <material name="White"/>
-        </visual>
-        <visual>
-            <origin xyz="-0.0225 0.0225 0.005" rpy="0 0 0"/>
-            <geometry>
-                <box size="0.015 0.015 0.002"/>
-            </geometry>
-            <material name="White"/>
-        </visual>
     </link>
-    <joint name="joint_camera_board_to_marker" type="fixed">
-        <parent link="camera_board"/>
+    <joint name="joint_sensor_board_to_marker" type="fixed">
+        <parent link="sensor_board"/>
         <child link="marker"/>
-        <origin xyz="0.01 0 0" rpy="0 0 0"/>
+        <origin xyz="0.30 0 0" rpy="0 0 0"/>
     </joint>
     <sensor_rplidar_a2 parent="sensor_board" prefix="lidar">

Commit message: Add option to have 2nd realsense camera in the rear

File: catkin_ws/src/car_robot_model/urdf/include/_d435.urdf.xacro (robot description, xacro)
@@ -7,5 +7,5 @@
 -->
 <robot name="sensor_d435" xmlns:xacro="http://ros.org/wiki/xacro">
-  <xacro:macro name="sensor_d435" params="parent *origin">
+  <xacro:macro name="sensor_d435" params="sensor_name parent *origin">
     <xacro:property name="M_PI" value="3.1415926535897931" />
     <!-- The following values are approximate, and the camera node
@@ -26,20 +26,20 @@
     <xacro:property name="d435_cam_depth_py" value="0.0175"/>
     <xacro:property name="d435_cam_depth_pz" value="${d435_cam_height/2}"/>
-    <material name="aluminum">
+    <material name="${sensor_name}aluminum">
       <color rgba="0.5 0.5 0.5 1"/>
     </material>
     <!-- camera body, with origin at bottom screw mount -->
-    <joint name="camera_joint" type="fixed">
+    <joint name="${sensor_name}_joint" type="fixed">
       <xacro:insert_block name="origin" />
       <parent link="${parent}"/>
-      <child link="camera_bottom_screw_frame" />
+      <child link="${sensor_name}_bottom_screw_frame" />
     </joint>
-    <link name="camera_bottom_screw_frame"/>
-    <joint name="camera_link_joint" type="fixed">
+    <link name="${sensor_name}_bottom_screw_frame"/>
+    <joint name="${sensor_name}_link_joint" type="fixed">
       <origin xyz="0 ${d435_cam_depth_py} ${d435_cam_depth_pz}" rpy="0 0 0"/>
-      <parent link="camera_bottom_screw_frame"/>
-      <child link="camera_link" />
+      <parent link="${sensor_name}_bottom_screw_frame"/>
+      <child link="${sensor_name}_link" />
     </joint>
-    <link name="camera_link">
+    <link name="${sensor_name}_link">
       <visual>
         <origin xyz="${d435_cam_mount_from_center_offset} ${-d435_cam_depth_py} 0" rpy="${M_PI/2} 0 ${M_PI/2}"/>
@@ -49,5 +49,5 @@
           <!--<mesh filename="package://realsense2_camera/meshes/d435/d435.dae" />-->
         </geometry>
-        <material name="aluminum"/>
+        <material name="${sensor_name}aluminum"/>
       </visual>
       <collision>
@@ -65,55 +65,55 @@
     </link>
     <!-- camera depth joints and links -->
-    <joint name="camera_depth_joint" type="fixed">
+    <joint name="${sensor_name}_depth_joint" type="fixed">
       <origin xyz="0 0 0" rpy="0 0 0"/>
-      <parent link="camera_link"/>
-      <child link="camera_depth_frame" />
+      <parent link="${sensor_name}_link"/>
+      <child link="${sensor_name}_depth_frame" />
     </joint>
-    <link name="camera_depth_frame"/>
-    <joint name="camera_depth_optical_joint" type="fixed">
+    <link name="${sensor_name}_depth_frame"/>
+    <joint name="${sensor_name}_depth_optical_joint" type="fixed">
       <origin xyz="0 0 0" rpy="${-M_PI/2} 0 ${-M_PI/2}" />
-      <parent link="camera_depth_frame" />
-      <child link="camera_depth_optical_frame" />
+      <parent link="${sensor_name}_depth_frame" />
+      <child link="${sensor_name}_depth_optical_frame" />
     </joint>
-    <link name="camera_depth_optical_frame"/>
+    <link name="${sensor_name}_depth_optical_frame"/>
     <!-- camera left IR joints and links -->
-    <joint name="camera_left_ir_joint" type="fixed">
+    <joint name="${sensor_name}_left_ir_joint" type="fixed">
       <origin xyz="0 ${d435_cam_depth_to_left_ir_offset} 0" rpy="0 0 0" />
-      <parent link="camera_depth_frame" />
-      <child link="camera_left_ir_frame" />
+      <parent link="${sensor_name}_depth_frame" />
+      <child link="${sensor_name}_left_ir_frame" />
     </joint>
-    <link name="camera_left_ir_frame"/>
-    <joint name="camera_left_ir_optical_joint" type="fixed">
+    <link name="${sensor_name}_left_ir_frame"/>
+    <joint name="${sensor_name}_left_ir_optical_joint" type="fixed">
       <origin xyz="0 0 0" rpy="${-M_PI/2} 0 ${-M_PI/2}" />
-      <parent link="camera_left_ir_frame" />
-      <child link="camera_left_ir_optical_frame" />
+      <parent link="${sensor_name}_left_ir_frame" />
+      <child link="${sensor_name}_left_ir_optical_frame" />
     </joint>
-    <link name="camera_left_ir_optical_frame"/>
+    <link name="${sensor_name}_left_ir_optical_frame"/>
     <!-- camera right IR joints and links -->
-    <joint name="camera_right_ir_joint" type="fixed">
+    <joint name="${sensor_name}_right_ir_joint" type="fixed">
       <origin xyz="0 ${d435_cam_depth_to_right_ir_offset} 0" rpy="0 0 0" />
-      <parent link="camera_depth_frame" />
-      <child link="camera_right_ir_frame" />
+      <parent link="${sensor_name}_depth_frame" />
+      <child link="${sensor_name}_right_ir_frame" />
     </joint>
-    <link name="camera_right_ir_frame"/>
-    <joint name="camera_right_ir_optical_joint" type="fixed">
+    <link name="${sensor_name}_right_ir_frame"/>
+    <joint name="${sensor_name}_right_ir_optical_joint" type="fixed">
       <origin xyz="0 0 0" rpy="${-M_PI/2} 0 ${-M_PI/2}" />
-      <parent link="camera_right_ir_frame" />
-      <child link="camera_right_ir_optical_frame" />
+      <parent link="${sensor_name}_right_ir_frame" />
+      <child link="${sensor_name}_right_ir_optical_frame" />
     </joint>
-    <link name="camera_right_ir_optical_frame"/>
+    <link name="${sensor_name}_right_ir_optical_frame"/>
     <!-- camera color joints and links -->
-    <joint name="camera_color_joint" type="fixed">
+    <joint name="${sensor_name}_color_joint" type="fixed">
       <origin xyz="0 ${d435_cam_depth_to_color_offset} 0" rpy="0 0 0" />
-      <parent link="camera_depth_frame" />
-      <child link="camera_color_frame" />
+      <parent link="${sensor_name}_depth_frame" />
+      <child link="${sensor_name}_color_frame" />
     </joint>
-    <link name="camera_color_frame"/>
-    <joint name="camera_color_optical_joint" type="fixed">
+    <link name="${sensor_name}_color_frame"/>
+    <joint name="${sensor_name}_color_optical_joint" type="fixed">
       <origin xyz="0 0 0" rpy="${-M_PI/2} 0 ${-M_PI/2}" />
-      <parent link="camera_color_frame" />
-      <child link="camera_color_optical_frame" />
+      <parent link="${sensor_name}_color_frame" />
+      <child link="${sensor_name}_color_optical_frame" />
     </joint>
-    <link name="camera_color_optical_frame"/>
+    <link name="${sensor_name}_color_optical_frame"/>
   </xacro:macro>
 </robot>
