Commit message: Add aruco marker

File: catkin_ws/src/car_robot_model/urdf/include/sensors.xacro (robot description, xacro)
@@ -112,7 +112,92 @@
         <origin xyz="-0.04 0 0" rpy="0 0 0"/>
     </joint>
-    <xacro:sensor_rplidar_a2 parent="sensor_board" prefix="lidar">
+    <!-- Aruco Marker -->
+    <link name="marker">
+        <inertial>
+            <mass value="0.2000000"/>
+            <origin xyz="0.00000000 0.00000000 0.00000000" rpy="0 0 0"/>
+            <inertia ixx="0.00000000" ixy="0.0" ixz="0.0"
+                     iyy="0.00000000" iyz="0.0"
+                     izz="0.00000000"/>
+        </inertial>
+        <visual>
+            <origin xyz="0 0 0.003" rpy="0 0 0"/>
+            <geometry>
+                <box size="0.12 0.12 0.002"/>
+            </geometry>
+            <material name="White"/>
+        </visual>
+        <visual>
+            <origin xyz="0.0 0.0 0.004" rpy="0 0 0"/>
+            <geometry>
+                <box size="0.09 0.09 0.002"/>
+            </geometry>
+            <material name="Black"/>
+        </visual>
+        <visual>
+            <origin xyz="0.0225 0.0225 0.005" rpy="0 0 0"/>
+            <geometry>
+                <box size="0.015 0.015 0.002"/>
+            </geometry>
+            <material name="White"/>
+        </visual>
+        <visual>
+            <origin xyz="0.0225 0.0075 0.005" rpy="0 0 0"/>
+            <geometry>
+                <box size="0.015 0.015 0.002"/>
+            </geometry>
+            <material name="White"/>
+        </visual>
+        <visual>
+            <origin xyz="0.0225 -0.0075 0.005" rpy="0 0 0"/>
+            <geometry>
+                <box size="0.015 0.015 0.002"/>
+            </geometry>
+            <material name="White"/>
+        </visual>
+        <visual>
+            <origin xyz="0.0075 0.0225 0.005" rpy="0 0 0"/>
+            <geometry>
+                <box size="0.015 0.015 0.002"/>
+            </geometry>
+            <material name="White"/>
+        </visual>
+        <visual>
+            <origin xyz="0.0075 -0.0075 0.005" rpy="0 0 0"/>
+            <geometry>
+                <box size="0.015 0.015 0.002"/>
+            </geometry>
+            <material name="White"/>
+        </visual>
+        <visual>
+            <origin xyz="0.0075 -0.0225 0.005" rpy="0 0 0"/>
+            <geometry>
+                <box size="0.015 0.015 0.002"/>
+            </geometry>
+            <material name="White"/>
+        </visual>
+        <visual>
+            <origin xyz="-0.0075 0.0075 0.005" rpy="0 0 0"/>
+            <geometry>
+                <box size="0.015 0.015 0.002"/>
+            </geometry>
+            <material name="White"/>
+        </visual>
+        <visual>
+            <origin xyz="-0.0225 0.0225 0.005" rpy="0 0 0"/>
+            <geometry>
+                <box size="0.015 0.015 0.002"/>
+            </geometry>
+            <material name="White"/>
+        </visual>
+    </link>
+    <joint name="joint_camera_board_to_marker" type="fixed">
+        <parent link="camera_board"/>
+        <child link="marker"/>
+        <origin xyz="0.01 0 0" rpy="0 0 0"/>
+    </joint>
+    <sensor_rplidar_a2 parent="sensor_board" prefix="lidar">
         <origin xyz="0.24 0 0" rpy="0 0 0"/>
-    </xacro:sensor_rplidar_a2>
+    </sensor_rplidar_a2>
     <!-- front camera -->
     <xacro:property name="front_camera_name" value="camera"/>

Commit message: Update sensors.xacro
Update lidar position

File: catkin_ws/src/car_robot_model/urdf/include/sensors.xacro (robot description, xacro)
@@ -198,5 +198,5 @@
     </joint>
     <sensor_rplidar_a2 parent="sensor_board" prefix="lidar">
-        <origin xyz="0.24 0 0" rpy="0 0 0"/>
+        <origin xyz="0.22 0 0" rpy="0 0 0"/>
     </sensor_rplidar_a2>
     <!-- front camera -->

Commit message: Update camera position

File: catkin_ws/src/car_robot_model/urdf/include/sensors.xacro (robot description, xacro)
@@ -57,5 +57,5 @@
         <parent link="sensor_board"/>
         <child link="camera_board"/>
-        <origin xyz="0.109 0 0.105" rpy="0 0 0"/>
+        <origin xyz="-0.07 0 0.15" rpy="0 0 0"/>
     </joint>
     <!--*************************************************-->
@@ -203,5 +203,5 @@
     <xacro:property name="front_camera_name" value="camera"/>
     <sensor_d435 parent="camera_board">
-        <origin xyz="0.087 0 0" rpy="0 0 0"/>
+        <origin xyz="0.087 0 0.04" rpy="0 0.15 0"/>
     </sensor_d435>
 </robot>

Commit message: Update autominy launch mappings

File: catkin_ws/src/car_robot_model/urdf/include/sensors.xacro (robot description, xacro)
@@ -198,5 +198,5 @@
     </joint>
     <sensor_rplidar_a2 parent="sensor_board" prefix="lidar">
-        <origin xyz="0.22 0 0" rpy="0 0 0"/>
+        <origin xyz="0.21 0 0" rpy="0 0 0"/>
     </sensor_rplidar_a2>
     <!-- front camera -->

Commit message: Remove imu rotation

File: catkin_ws/src/car_robot_model/urdf/include/sensors.xacro (robot description, xacro)
@@ -88,5 +88,5 @@
         <parent link="sensor_board"/>
         <child link="imu"/>
-        <origin xyz="0.035 -0.035 0.0025" rpy="0 0 ${PI/2}"/>
+        <origin xyz="0.035 -0.035 0.0025" rpy="0 0 0"/>
     </joint>
     <!-- Odroid -->

Commit message: Add IMU frame

File: catkin_ws/src/car_robot_model/urdf/include/sensors.xacro (robot description, xacro)
@@ -90,4 +90,12 @@
         <origin xyz="0.035 -0.035 0.0025" rpy="0 0 0"/>
     </joint>
+    <!-- BNO055 -->
+    <link name="bno055">
+    </link>
+    <joint name="joint_sensor_board_to_imu" type="fixed">
+        <parent link="sensor_board"/>
+        <child link="bno055"/>
+        <origin xyz="0.235 0.0 0.023" rpy="0 0 0"/>
+    </joint>
     <!-- Odroid -->
     <link name="odroid">

Commit message: Fix joint name

File: catkin_ws/src/car_robot_model/urdf/include/sensors.xacro (robot description, xacro)
@@ -93,5 +93,5 @@
     <link name="bno055">
     </link>
-    <joint name="joint_sensor_board_to_imu" type="fixed">
+    <joint name="joint_sensor_board_to_bno055" type="fixed">
         <parent link="sensor_board"/>
         <child link="bno055"/>

Commit message: Fix bno055 rotation

File: catkin_ws/src/car_robot_model/urdf/include/sensors.xacro (robot description, xacro)
@@ -96,5 +96,5 @@
         <parent link="sensor_board"/>
         <child link="bno055"/>
-        <origin xyz="0.235 0.0 0.023" rpy="0 0 0"/>
+        <origin xyz="0.235 0.0 0.023" rpy="0 0 1.5708"/>
     </joint>
     <!-- Odroid -->

Commit message: Add 2nd realsense camera to urdf

File: catkin_ws/src/car_robot_model/urdf/include/sensors.xacro (robot description, xacro)
@@ -133,6 +133,9 @@
     <!-- front camera -->
     <xacro:property name="front_camera_name" value="camera"/>
-    <sensor_d435 parent="camera_board">
+    <sensor_d435 parent="camera_board" sensor_name="camera">
         <origin xyz="0.087 0 0.04" rpy="0 0.15 0"/>
     </sensor_d435>
+    <sensor_d435 parent="camera_board" sensor_name="rear_camera">
+        <origin xyz="0 0 1.57" rpy="0 0.15 0"/>
+    </sensor_d435>
 </robot>

Commit message: Fix rear camera position

File: catkin_ws/src/car_robot_model/urdf/include/sensors.xacro (robot description, xacro)
@@ -137,5 +137,5 @@
     </sensor_d435>
     <sensor_d435 parent="camera_board" sensor_name="rear_camera">
-        <origin xyz="0 0 1.57" rpy="0 0.15 0"/>
+        <origin xyz="0 0 0" rpy="0 0.15 3.141"/>
     </sensor_d435>
 </robot>
