Commit message: Update lidar and realsense camera

File: catkin_ws/src/car_robot_model/urdf/car.xacro (robot description, xacro)
@@ -1,7 +1,7 @@
 <?xml version="1.0"?>
-<robot name="model_car" xmlns:xacro="http://www.ros.org/wiki/xacro">
-  <!-- Included URDF Files -->
-  <xacro:include filename="$(find car_robot_model)/urdf/include/materials.xacro" />
-  <xacro:include filename="$(find car_robot_model)/urdf/include/platform.xacro" />
-  <xacro:include filename="$(find car_robot_model)/urdf/include/sensors.xacro" />
+<robot xmlns:xacro="http://www.ros.org/wiki/xacro" name="model_car">
+    <!-- Included URDF Files -->
+    <xacro:include filename="$(find car_robot_model)/urdf/include/materials.xacro"/>
+    <xacro:include filename="$(find car_robot_model)/urdf/include/platform.xacro"/>
+    <xacro:include filename="$(find car_robot_model)/urdf/include/sensors.xacro"/>
 </robot>

File: catkin_ws/src/car_robot_model/urdf/include/platform.xacro (robot description, xacro)
@@ -1,251 +1,251 @@
 <?xml version="1.0"?>
-<robot name="model_car" xmlns:xacro="http://www.ros.org/wiki/xacro">
-  <xacro:property name="PI" value="3.1415926535897931" />
-  <xacro:property name="angle_limit" value="${PI/3.0}" />
-  <xacro:property name="wheel_width" value="0.001" />
-  <link name="base_link">
-  </link>
-  <link name="body">
-    <inertial>
-      <mass value="6" />
-      <origin xyz="0.15971917 0.00000000 0.00197764" />
-      <inertia ixx="0.0067970" ixy="0.0" ixz="-0.0008808"
-               iyy="0.0784672" iyz="0.0"
-               izz="0.0838770" />
-    </inertial>
-    <visual>
-      <origin xyz="0 0 0" rpy="0 0 0" />
-      <geometry>
-        <mesh filename="package://car_robot_model/meshes/chassis.stl"/>
-      </geometry>
-      <material name="Black" />
-    </visual>
-    <collision>
-      <origin xyz="0 0 0" rpy="0 0 0" />
-      <geometry>
-        <mesh filename="package://car_robot_model/meshes/chassis.stl"/>
-      </geometry>
-    </collision>
-  </link>
-  <joint name="base_link_to_body" type="fixed">
-    <origin xyz="0.0 0 0.005" rpy="0 0 0" />
-    <parent link="base_link" />
-    <child link="body" />
-  </joint>
-  <joint name="base_link_rear_left_wheel_joint" type="revolute">
-    <origin xyz="0.0 -0.0825 0.03" rpy="${PI/2.0} 0 0" />
-    <axis xyz="0 0 1" />
-    <anchor xyz="0 0 0" />
-    <parent link="base_link" />
-    <child link="rear_left_wheel_link" />
-    <limit lower="-1000000000000.0" upper="1000000000000.0" effort="3.0" velocity="124"/>
-  </joint>
-  <transmission name="tran_rear_left">
-    <type>transmission_interface/SimpleTransmission</type>
-    <joint name="base_link_rear_left_wheel_joint">
-      <hardwareInterface>hardware_interface/EffortJointInterface</hardwareInterface>
-    </joint>
-    <actuator name="rear_left_motor">
-      <hardwareInterface>hardware_interface/EffortJointInterface</hardwareInterface>
-      <mechanicalReduction>1</mechanicalReduction>
-    </actuator>
-  </transmission>
-  <link name="rear_left_wheel_link">
-    <inertial>
-      <mass value="1" />
-      <origin xyz="0 0 0" rpy="0 0 0" />
-      <inertia  ixx="0.0002946" ixy="0.0" ixz="0.0"
-                iyy="0.0002946" iyz="0.0"
-                izz="0.000494" />
-    </inertial>
-    <visual>
-      <origin xyz="0 0 0" rpy="0 0 0" />
-      <geometry>
-        <mesh filename="package://car_robot_model/meshes/wheel.stl"/>
-      </geometry>
-      <material name="Black" />
-    </visual>
-    <collision>
-      <origin xyz="0 0 0" rpy="0 0 0" />
-      <geometry>
-        <cylinder radius="0.0315" length="${wheel_width}"/>
-      </geometry>
-    </collision>
-  </link>
-  <joint name="base_link_rear_right_wheel_joint" type="revolute">
-    <origin xyz="0.0 0.0825 0.03" rpy="-${PI/2.0} 0 0" />
-    <axis xyz="0 0 1" />
-    <anchor xyz="0 0 0" />
-    <parent link="base_link" />
-    <child link="rear_right_wheel_link" />
-    <limit lower="-1000000000000.0" upper="1000000000000.0" effort="3.0" velocity="124"/>
-  </joint>
-  <transmission name="tran_rear_right">
-    <type>transmission_interface/SimpleTransmission</type>
-    <joint name="base_link_rear_right_wheel_joint">
-      <hardwareInterface>hardware_interface/EffortJointInterface</hardwareInterface>
-    </joint>
-    <actuator name="rear_right_motor">
-      <hardwareInterface>hardware_interface/EffortJointInterface</hardwareInterface>
-      <mechanicalReduction>1</mechanicalReduction>
-    </actuator>
-  </transmission>
-  <link name="rear_right_wheel_link">
-    <inertial>
-      <mass value="1" />
-      <origin xyz="0 0 0" rpy="0 0 0" />
-      <inertia  ixx="0.0002946" ixy="0.0" ixz="0.0"
-                iyy="0.0002946" iyz="0.0"
-                izz="0.0004940" />
-    </inertial>
-    <visual>
-      <origin xyz="0 0 0" rpy="0 0 0" />
-      <geometry>
-        <mesh filename="package://car_robot_model/meshes/wheel.stl"/>
-      </geometry>
-      <material name="Black" />
-    </visual>
-    <collision>
-      <origin xyz="0 0 0" rpy="0 0 0" />
-      <geometry>
-        <cylinder radius="0.0315" length="${wheel_width}"/>
-      </geometry>
-    </collision>
-  </link>
-  <joint name="base_link_front_left_axel_joint" type="revolute">
-    <origin xyz="0.260 -0.0825 0.03" rpy="${PI/2.0} 0 0" />
-    <axis xyz="0 1 0" />
-    <anchor xyz="0 0 0" />
-    <parent link="base_link" />
-    <child link="front_left_axel_link" />
-    <limit lower="-${angle_limit}" upper="${angle_limit}" effort="9.6" velocity="5.3"/>
-    <dynamics damping="0.2"/>
-  </joint>
-  <transmission name="tran_front_left_axel">
-    <type>transmission_interface/SimpleTransmission</type>
-    <joint name="base_link_front_left_axel_joint">
-      <hardwareInterface>hardware_interface/EffortJointInterface</hardwareInterface>
-    </joint>
-    <actuator name="front_left_axel_motor">
-      <hardwareInterface>hardware_interface/EffortJointInterface</hardwareInterface>
-      <mechanicalReduction>1</mechanicalReduction>
-    </actuator>
-  </transmission>
-  <link name="front_left_axel_link">
-    <inertial>
-      <mass value="0.001" />
-      <origin xyz="0 0 0" rpy="0 0 0" />
-      <inertia  ixx="0.00001" ixy="0.0" ixz="0.0"
-                iyy="0.00001" iyz="0.0"
-                izz="0.00001" />
-    </inertial>
-  </link>
-  <joint name="front_left_axel_front_left_wheel_joint" type="revolute">
-    <origin xyz="0.0 0.0 0" rpy="0 0 0" />
-    <axis xyz="0 0 1" />
-    <anchor xyz="0 0 0" />
-    <parent link="front_left_axel_link" />
-    <child link="front_left_wheel_link" />
-    <limit lower="-1000000000000.0" upper="1000000000000.0" effort="3.0" velocity="124"/>
-  </joint>
-  <transmission name="tran_front_left_wheel">
-    <type>transmission_interface/SimpleTransmission</type>
-    <joint name="front_left_axel_front_left_wheel_joint">
-      <hardwareInterface>hardware_interface/EffortJointInterface</hardwareInterface>
-    </joint>
-    <actuator name="front_left_wheel_motor">
-      <hardwareInterface>hardware_interface/EffortJointInterface</hardwareInterface>
-      <mechanicalReduction>1</mechanicalReduction>
-    </actuator>
-  </transmission>
-  <link name="front_left_wheel_link">
-    <inertial>
-      <mass value="1" />
-      <origin xyz="0 0 0" rpy="0 0 0" />
-      <inertia  ixx="0.0002946" ixy="0.0" ixz="0.0"
-                iyy="0.0002946" iyz="0.0"
-                izz="0.0004940" />
-    </inertial>
-    <visual>
-      <origin xyz="0 0 0" rpy="0 0 0" />
-      <geometry>
-        <mesh filename="package://car_robot_model/meshes/wheel.stl"/>
-      </geometry>
-      <material name="Black" />
-    </visual>
-    <collision>
-      <origin xyz="0 0 0" rpy="0 0 0" />
-      <geometry>
-        <cylinder radius="0.0315" length="${wheel_width}"/>
-      </geometry>
-    </collision>
-  </link>
-  <joint name="base_link_front_right_axel_joint" type="revolute">
-    <origin xyz="0.260 0.0825 0.03" rpy="-${PI/2.0} 0 0" />
-    <axis xyz="0 1 0" />
-    <anchor xyz="0 0 0" />
-    <parent link="base_link" />
-    <child link="front_right_axel_link" />
-    <limit lower="-${angle_limit}" upper="${angle_limit}" effort="9.6" velocity="5.3"/>
-    <dynamics damping="0.2"/>
-  </joint>
-  <transmission name="tran_front_right_axel">
-    <type>transmission_interface/SimpleTransmission</type>
-    <joint name="base_link_front_right_axel_joint">
-      <hardwareInterface>hardware_interface/EffortJointInterface</hardwareInterface>
-    </joint>
-    <actuator name="front_right_axel_motor">
-      <hardwareInterface>hardware_interface/EffortJointInterface</hardwareInterface>
-      <mechanicalReduction>1</mechanicalReduction>
-    </actuator>
-  </transmission>
-  <link name="front_right_axel_link">
-    <inertial>
-      <mass value="0.001" />
-      <origin xyz="0 0 0" rpy="0 0 0" />
-      <inertia  ixx="0.00001" ixy="0.0" ixz="0.0"
-                iyy="0.00001" iyz="0.0"
-                izz="0.00001" />
-    </inertial>
-  </link>
-  <joint name="front_right_axel_front_right_wheel_joint" type="continuous">
-    <origin xyz="0.0 0.0 0" rpy="0 0 0" />
-    <axis xyz="0 0 1" />
-    <anchor xyz="0 0 0" />
-    <parent link="front_right_axel_link" />
-    <child link="front_right_wheel_link" />
-    <limit lower="-1000000000000.0" upper="1000000000000.0" effort="3.0" velocity="124"/>
-  </joint>
-  <transmission name="tran_front_right_wheel">
-    <type>transmission_interface/SimpleTransmission</type>
-    <joint name="front_right_axel_front_right_wheel_joint">
-      <hardwareInterface>hardware_interface/EffortJointInterface</hardwareInterface>
-    </joint>
-    <actuator name="front_right_wheel_motor">
-      <hardwareInterface>hardware_interface/EffortJointInterface</hardwareInterface>
-      <mechanicalReduction>1</mechanicalReduction>
-    </actuator>
-  </transmission>
-  <link name="front_right_wheel_link">
-    <inertial>
-      <mass value="1" />
-      <origin xyz="0 0 0" rpy="0 0 0" />
-      <inertia  ixx="0.0002946" ixy="0.0" ixz="0.0"
-                iyy="0.0002946" iyz="0.0"
-                izz="0.0004940" />
-    </inertial>
-    <visual>
-      <origin xyz="0 0 0" rpy="0 0 0" />
-      <geometry>
-        <mesh filename="package://car_robot_model/meshes/wheel.stl"/>
-      </geometry>
-      <material name="Black" />
-    </visual>
-    <collision>
-      <origin xyz="0 0 0" rpy="0 0 0" />
-      <geometry>
-        <cylinder radius="0.0315" length="${wheel_width}"/>
-      </geometry>
-    </collision>
-  </link>
+<robot xmlns:xacro="http://www.ros.org/wiki/xacro" name="model_car">
+    <xacro:property name="PI" value="3.1415926535897931"/>
+    <xacro:property name="angle_limit" value="${PI/3.0}"/>
+    <xacro:property name="wheel_width" value="0.001"/>
+    <link name="base_link">
+    </link>
+    <link name="body">
+        <inertial>
+            <mass value="6"/>
+            <origin xyz="0.15971917 0.00000000 0.00197764"/>
+            <inertia ixx="0.0067970" ixy="0.0" ixz="-0.0008808"
+                     iyy="0.0784672" iyz="0.0"
+                     izz="0.0838770"/>
+        </inertial>
+        <visual>
+            <origin xyz="0 0 0" rpy="0 0 0"/>
+            <geometry>
+                <mesh filename="package://car_robot_model/meshes/chassis.stl"/>
+            </geometry>
+            <material name="Black"/>
+        </visual>
+        <collision>
+            <origin xyz="0 0 0" rpy="0 0 0"/>
+            <geometry>
+                <mesh filename="package://car_robot_model/meshes/chassis.stl"/>
+            </geometry>
+        </collision>
+    </link>
+    <joint name="base_link_to_body" type="fixed">
+        <origin xyz="0.0 0 0.005" rpy="0 0 0"/>
+        <parent link="base_link"/>
+        <child link="body"/>
+    </joint>
+    <joint name="base_link_rear_left_wheel_joint" type="revolute">
+        <origin xyz="0.0 -0.0825 0.03" rpy="${PI/2.0} 0 0"/>
+        <axis xyz="0 0 1"/>
+        <anchor xyz="0 0 0"/>
+        <parent link="base_link"/>
+        <child link="rear_left_wheel_link"/>
+        <limit lower="-1000000000000.0" upper="1000000000000.0" effort="3.0" velocity="124"/>
+    </joint>
+    <transmission name="tran_rear_left">
+        <type>transmission_interface/SimpleTransmission</type>
+        <joint name="base_link_rear_left_wheel_joint">
+            <hardwareInterface>hardware_interface/EffortJointInterface</hardwareInterface>
+        </joint>
+        <actuator name="rear_left_motor">
+            <hardwareInterface>hardware_interface/EffortJointInterface</hardwareInterface>
+            <mechanicalReduction>1</mechanicalReduction>
+        </actuator>
+    </transmission>
+    <link name="rear_left_wheel_link">
+        <inertial>
+            <mass value="1"/>
+            <origin xyz="0 0 0" rpy="0 0 0"/>
+            <inertia ixx="0.0002946" ixy="0.0" ixz="0.0"
+                     iyy="0.0002946" iyz="0.0"
+                     izz="0.000494"/>
+        </inertial>
+        <visual>
+            <origin xyz="0 0 0" rpy="0 0 0"/>
+            <geometry>
+                <mesh filename="package://car_robot_model/meshes/wheel.stl"/>
+            </geometry>
+            <material name="Black"/>
+        </visual>
+        <collision>
+            <origin xyz="0 0 0" rpy="0 0 0"/>
+            <geometry>
+                <cylinder radius="0.0315" length="${wheel_width}"/>
+            </geometry>
+        </collision>
+    </link>
+    <joint name="base_link_rear_right_wheel_joint" type="revolute">
+        <origin xyz="0.0 0.0825 0.03" rpy="-${PI/2.0} 0 0"/>
+        <axis xyz="0 0 1"/>
+        <anchor xyz="0 0 0"/>
+        <parent link="base_link"/>
+        <child link="rear_right_wheel_link"/>
+        <limit lower="-1000000000000.0" upper="1000000000000.0" effort="3.0" velocity="124"/>
+    </joint>
+    <transmission name="tran_rear_right">
+        <type>transmission_interface/SimpleTransmission</type>
+        <joint name="base_link_rear_right_wheel_joint">
+            <hardwareInterface>hardware_interface/EffortJointInterface</hardwareInterface>
+        </joint>
+        <actuator name="rear_right_motor">
+            <hardwareInterface>hardware_interface/EffortJointInterface</hardwareInterface>
+            <mechanicalReduction>1</mechanicalReduction>
+        </actuator>
+    </transmission>
+    <link name="rear_right_wheel_link">
+        <inertial>
+            <mass value="1"/>
+            <origin xyz="0 0 0" rpy="0 0 0"/>
+            <inertia ixx="0.0002946" ixy="0.0" ixz="0.0"
+                     iyy="0.0002946" iyz="0.0"
+                     izz="0.0004940"/>
+        </inertial>
+        <visual>
+            <origin xyz="0 0 0" rpy="0 0 0"/>
+            <geometry>
+                <mesh filename="package://car_robot_model/meshes/wheel.stl"/>
+            </geometry>
+            <material name="Black"/>
+        </visual>
+        <collision>
+            <origin xyz="0 0 0" rpy="0 0 0"/>
+            <geometry>
+                <cylinder radius="0.0315" length="${wheel_width}"/>
+            </geometry>
+        </collision>
+    </link>
+    <joint name="base_link_front_left_axel_joint" type="revolute">
+        <origin xyz="0.260 -0.0825 0.03" rpy="${PI/2.0} 0 0"/>
+        <axis xyz="0 1 0"/>
+        <anchor xyz="0 0 0"/>
+        <parent link="base_link"/>
+        <child link="front_left_axel_link"/>
+        <limit lower="-${angle_limit}" upper="${angle_limit}" effort="9.6" velocity="5.3"/>
+        <dynamics damping="0.2"/>
+    </joint>
+    <transmission name="tran_front_left_axel">
+        <type>transmission_interface/SimpleTransmission</type>
+        <joint name="base_link_front_left_axel_joint">
+            <hardwareInterface>hardware_interface/EffortJointInterface</hardwareInterface>
+        </joint>
+        <actuator name="front_left_axel_motor">
+            <hardwareInterface>hardware_interface/EffortJointInterface</hardwareInterface>
+            <mechanicalReduction>1</mechanicalReduction>
+        </actuator>
+    </transmission>
+    <link name="front_left_axel_link">
+        <inertial>
+            <mass value="0.001"/>
+            <origin xyz="0 0 0" rpy="0 0 0"/>
+            <inertia ixx="0.00001" ixy="0.0" ixz="0.0"
+                     iyy="0.00001" iyz="0.0"
+                     izz="0.00001"/>
+        </inertial>
+    </link>
+    <joint name="front_left_axel_front_left_wheel_joint" type="revolute">
+        <origin xyz="0.0 0.0 0" rpy="0 0 0"/>
+        <axis xyz="0 0 1"/>
+        <anchor xyz="0 0 0"/>
+        <parent link="front_left_axel_link"/>
+        <child link="front_left_wheel_link"/>
+        <limit lower="-1000000000000.0" upper="1000000000000.0" effort="3.0" velocity="124"/>
+    </joint>
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