Commit message: Update lidar and realsense camera

File: catkin_ws/src/car_robot_model/urdf/include/sensors.xacro (robot description, xacro)
@@ -1,212 +1,122 @@
 <?xml version="1.0"?>
-<robot name="model_car" xmlns:xacro="http://www.ros.org/wiki/xacro">
-  <!-- Included URDF Files -->
-  <xacro:property name="PI" value="3.1415926535897931" />
-  <link name="sensor_board">
-    <inertial>
-      <mass value="6" />
-      <origin xyz="0.12043628 0.00000000 0.00171950" rpy="0 0 0"/>
-      <inertia ixx="0.0123739" ixy="0.0" ixz="0.0003463"
-               iyy="0.0711051" iyz="0.0"
-               izz="0.0820107" />
-    </inertial>
-    <visual>
-      <origin xyz="0.0 0.0 0.0" rpy="0 0 0"/>
-      <geometry>
-        <mesh filename="package://car_robot_model/meshes/sensor_board.stl" />
-      </geometry>
-      <material name="Grey" />
-    </visual>
-    <collision>
-      <origin xyz="0.0 0.0 0.0" rpy="0 0 0"/>
-      <geometry>
-        <mesh filename="package://car_robot_model/meshes/sensor_board.stl" />
-      </geometry>
-    </collision>
-  </link>
-  <joint name="joint_base_link_to_sensor_board" type="fixed" >
-    <parent link="base_link"/>
-    <child link="sensor_board"/>
-    <origin xyz="0 0 0.07" rpy="0 0 0"/>
-  </joint>
-  <link name="camera_board">
-    <inertial>
-      <mass value="0.6000000" />
-      <origin xyz="0.04901990 0.00000000 0.00000000" rpy="0 0 0"/>
-      <inertia ixx="0.0003816" ixy="0.0" ixz="0.0"
-               iyy="0.0003420" iyz="0.0"
-               izz="0.0007211" />
-    </inertial>
-    <visual>
-      <origin xyz="0.0 0.0 0.0" rpy="0 0 0"/>
-      <geometry>
-        <mesh filename="package://car_robot_model/meshes/camera_board.stl" />
-      </geometry>
-      <material name="Grey" />
-    </visual>
-    <collision>
-      <origin xyz="0.0 0.0 0.0" rpy="0 0 0"/>
-      <geometry>
-        <mesh filename="package://car_robot_model/meshes/camera_board.stl" />
-      </geometry>
-    </collision>
-  </link>
-  <joint name="joint_sensor_board_to_camera_board" type="fixed" >
-    <parent link="sensor_board"/>
-    <child link="camera_board"/>
-    <origin xyz="0.109 0 0.105" rpy="0 0 0"/>
-  </joint>
-  <!--*************************************************-->
-  <!--*               Sensors                         *-->
-  <!--*************************************************-->
-  <!-- IMU -->
-  <link name="imu">
-    <inertial>
-      <mass value="0.0200000" />
-      <origin xyz="0.00000000 0.00000000 0.00150000" rpy="0 0 0"/>
-      <inertia ixx="0.0000007" ixy="0.0" ixz="0.0"
-               iyy="0.0000004" iyz="0.0"
-               izz="0.0000011" />
-    </inertial>
-    <visual>
-      <origin xyz="0 0 0" rpy="0 0 0"/>
-      <geometry>
-        <mesh filename="package://car_robot_model/meshes/IMU.stl" />
-      </geometry>
-      <material name="Black" />
-    </visual>
-    <collision>
-      <origin xyz="0 0 0" rpy="0 0 0"/>
-      <geometry>
-        <mesh filename="package://car_robot_model/meshes/IMU.stl" />
-      </geometry>
-    </collision>
-  </link>
-  <joint name="joint_sensor_board_to_imu" type="fixed" >
-    <parent link="sensor_board"/>
-    <child link="imu"/>
-    <origin xyz="0.035 -0.035 0.0025" rpy="0 0 ${PI/2}"/>
-  </joint>
-  <!-- Odroid -->
-  <link name="odroid">
-    <inertial>
-      <mass value="0.2000000" />
-      <origin xyz="0.00000000 0.00000000 0.00000000" rpy="0 0 0"/>
-      <inertia ixx="0.00000000" ixy="0.0" ixz="0.0"
-               iyy="0.00000000" iyz="0.0"
-               izz="0.00000000" />
-    </inertial>
-    <visual>
-      <origin xyz="0 0 0.01" rpy="0 0 0" />
-      <geometry>
-        <box size="0.06 0.08 0.015" />
-      </geometry>
-      <material name="Black" />
-    </visual>
-  </link>
-  <joint name="joint_sensor_board_to_odroid" type="fixed" >
-    <parent link="sensor_board"/>
-    <child link="odroid"/>
-    <origin xyz="-0.04 0 0" rpy="0 0 0"/>
-  </joint>
-  <!-- RP_LIDAR -->
-  <link name="laser">
-    <inertial>
-      <mass value="1.8362923" />
-      <origin xyz="0.0000000 0.0000000 -0.01040000" rpy="0 0 0"/>
-      <inertia ixx="0.0009124" ixy="0.0" ixz="0.0"
-               iyy="0.0009124" iyz="0.0"
-               izz="0.0013154" />
-    </inertial>
-    <visual>
-      <origin xyz="0 0 0" rpy="0 0 0"/>
-      <geometry>
-        <mesh filename="package://car_robot_model/meshes/RP-LIDAR.stl" />
-      </geometry>
-      <material name="Black" />
-    </visual>
-    <collision>
-      <origin xyz="0 0 0" rpy="0 0 0"/>
-      <geometry>
-        <mesh filename="package://car_robot_model/meshes/RP-LIDAR.stl" />
-      </geometry>
-    </collision>
-  </link>
-  <joint name="joint_sensor_board_to_laser" type="fixed" >
-    <parent link="sensor_board"/>
-    <child link="laser"/>
-    <origin xyz="0.25 0 0.0333" rpy="0 0 0"/>
-  </joint>
-  <!-- top camera -->
-  <!--  <xacro:property name="top_camera_name" value="top_camera" />-->
-  <link name="top_camera">
-    <inertial>
-      <mass value="0.1600000" />
-      <origin xyz="0.00000000 0.00000000 -0.01396703" rpy="0 0 0"/>
-      <inertia ixx="0.0000170" ixy="0.0" ixz="0.0"
-               iyy="0.0000170" iyz="0.0"
-               izz="0.0000183" />
-    </inertial>
-    <visual>
-      <origin xyz="0 0 0" rpy="0 ${PI/2} 0"/>
-      <geometry>
-        <mesh filename="package://car_robot_model/meshes/gps_camera.stl" />
-      </geometry>
-      <material name="Black" />
-    </visual>
-    <collision>
-      <origin xyz="0 0 0" rpy="0 ${PI/2} 0"/>
-      <geometry>
-        <mesh filename="package://car_robot_model/meshes/gps_camera.stl" />
-      </geometry>
-    </collision>
-  </link>
-  <joint name="joint_camera_board_to_top_camera" type="fixed" >
-    <parent link="camera_board"/>
-    <child link="top_camera"/>
-    <origin xyz="0.019 0 0.0405" rpy="0 -${PI/2} ${PI}"/>
-  </joint>
-  <link name="top_camera_optical">
-  </link>
-  <joint name="joint_top_camera_to_top_camera_optical" type="fixed" >
-    <parent link="top_camera"/>
-    <child link="top_camera_optical"/>
-    <origin xyz="0.0 0 0.0" rpy="-${PI/2} 0 -${PI/2}"/>
-  </joint>
-  <!-- front camera -->
-  <xacro:property name="front_camera_name" value="camera" />
-  <link name="${front_camera_name}_link">
-    <inertial>
-      <mass value="1.3000000" />
-      <origin xyz="0.00000000 0.00000000 -0.01150000" rpy="0 0 0"/>
-      <inertia ixx="0.0017500" ixy="0.0" ixz="0.0"
-               iyy="0.0001146" iyz="0.0"
-               izz="0.0017500" />
-    </inertial>
-    <visual>
-      <origin xyz="0 0 0" rpy="0 0 0"/>
-      <geometry>
-        <mesh filename="package://car_robot_model/meshes/creative_camera.stl" />
-      </geometry>
-      <material name="Black" />
-    </visual>
-    <collision>
-      <origin xyz="0 0 0" rpy="0 0 0"/>
-      <geometry>
-        <mesh filename="package://car_robot_model/meshes/creative_camera.stl" />
-      </geometry>
-    </collision>
-  </link>
-  <joint name="joint_camera_board_to_${front_camera_name}_link" type="fixed" >
-    <parent link="camera_board"/>
-    <child link="${front_camera_name}_link"/>
-    <origin xyz="0.119 0 0.0" rpy="0 0 0"/>
-  </joint>
-  <link name="${front_camera_name}_rgb_optical_frame">
-  </link>
-  <joint name="joint_${front_camera_name}_link_to_${front_camera_name}_rgb_optical_frame" type="fixed" >
-    <parent link="${front_camera_name}_link"/>
-    <child link="${front_camera_name}_rgb_optical_frame"/>
-    <origin xyz="0 0 0" rpy="-${PI/2} 0 -${PI/2}"/>
-  </joint>
+<robot xmlns:xacro="http://www.ros.org/wiki/xacro" name="model_car">
+    <!-- Included URDF Files -->
+    <xacro:include filename="$(find car_robot_model)/urdf/include/rplidar_a2.xacro"/>
+    <xacro:include filename="$(find realsense2_camera)/urdf/_d435.urdf.xacro"/>
+    <xacro:property name="PI" value="3.1415926535897931"/>
+    <link name="sensor_board">
+        <inertial>
+            <mass value="6"/>
+            <origin xyz="0.12043628 0.00000000 0.00171950" rpy="0 0 0"/>
+            <inertia ixx="0.0123739" ixy="0.0" ixz="0.0003463"
+                     iyy="0.0711051" iyz="0.0"
+                     izz="0.0820107"/>
+        </inertial>
+        <visual>
+            <origin xyz="0.0 0.0 0.0" rpy="0 0 0"/>
+            <geometry>
+                <mesh filename="package://car_robot_model/meshes/sensor_board.stl"/>
+            </geometry>
+            <material name="Grey"/>
+        </visual>
+        <collision>
+            <origin xyz="0.0 0.0 0.0" rpy="0 0 0"/>
+            <geometry>
+                <mesh filename="package://car_robot_model/meshes/sensor_board.stl"/>
+            </geometry>
+        </collision>
+    </link>
+    <joint name="joint_base_link_to_sensor_board" type="fixed">
+        <parent link="base_link"/>
+        <child link="sensor_board"/>
+        <origin xyz="0 0 0.07" rpy="0 0 0"/>
+    </joint>
+    <link name="camera_board">
+        <inertial>
+            <mass value="0.6000000"/>
+            <origin xyz="0.04901990 0.00000000 0.00000000" rpy="0 0 0"/>
+            <inertia ixx="0.0003816" ixy="0.0" ixz="0.0"
+                     iyy="0.0003420" iyz="0.0"
+                     izz="0.0007211"/>
+        </inertial>
+        <visual>
+            <origin xyz="0.0 0.0 0.0" rpy="0 0 0"/>
+            <geometry>
+                <mesh filename="package://car_robot_model/meshes/camera_board.stl"/>
+            </geometry>
+            <material name="Grey"/>
+        </visual>
+        <collision>
+            <origin xyz="0.0 0.0 0.0" rpy="0 0 0"/>
+            <geometry>
+                <mesh filename="package://car_robot_model/meshes/camera_board.stl"/>
+            </geometry>
+        </collision>
+    </link>
+    <joint name="joint_sensor_board_to_camera_board" type="fixed">
+        <parent link="sensor_board"/>
+        <child link="camera_board"/>
+        <origin xyz="0.109 0 0.105" rpy="0 0 0"/>
+    </joint>
+    <!--*************************************************-->
+    <!--*               Sensors                         *-->
+    <!--*************************************************-->
+    <!-- IMU -->
+    <link name="imu">
+        <inertial>
+            <mass value="0.0200000"/>
+            <origin xyz="0.00000000 0.00000000 0.00150000" rpy="0 0 0"/>
+            <inertia ixx="0.0000007" ixy="0.0" ixz="0.0"
+                     iyy="0.0000004" iyz="0.0"
+                     izz="0.0000011"/>
+        </inertial>
+        <visual>
+            <origin xyz="0 0 0" rpy="0 0 0"/>
+            <geometry>
+                <mesh filename="package://car_robot_model/meshes/IMU.stl"/>
+            </geometry>
+            <material name="Black"/>
+        </visual>
+        <collision>
+            <origin xyz="0 0 0" rpy="0 0 0"/>
+            <geometry>
+                <mesh filename="package://car_robot_model/meshes/IMU.stl"/>
+            </geometry>
+        </collision>
+    </link>
+    <joint name="joint_sensor_board_to_imu" type="fixed">
+        <parent link="sensor_board"/>
+        <child link="imu"/>
+        <origin xyz="0.035 -0.035 0.0025" rpy="0 0 ${PI/2}"/>
+    </joint>
+    <!-- Odroid -->
+    <link name="odroid">
+        <inertial>
+            <mass value="0.2000000"/>
+            <origin xyz="0.00000000 0.00000000 0.00000000" rpy="0 0 0"/>
+            <inertia ixx="0.00000000" ixy="0.0" ixz="0.0"
+                     iyy="0.00000000" iyz="0.0"
+                     izz="0.00000000"/>
+        </inertial>
+        <visual>
+            <origin xyz="0 0 0.01" rpy="0 0 0"/>
+            <geometry>
+                <box size="0.06 0.08 0.015"/>
+            </geometry>
+            <material name="Black"/>
+        </visual>
+    </link>
+    <joint name="joint_sensor_board_to_odroid" type="fixed">
+        <parent link="sensor_board"/>
+        <child link="odroid"/>
+        <origin xyz="-0.04 0 0" rpy="0 0 0"/>
+    </joint>
+    <xacro:sensor_rplidar_a2 parent="sensor_board" prefix="lidar">
+        <origin xyz="0.24 0 0" rpy="0 0 0"/>
+    </xacro:sensor_rplidar_a2>
+    <!-- front camera -->
+    <xacro:property name="front_camera_name" value="camera"/>
+    <sensor_d435 parent="camera_board">
+        <origin xyz="0.087 0 0" rpy="0 0 0"/>
+    </sensor_d435>
 </robot>
