Commit message: Try to align to base_link

File: catkin_ws/src/autominy_simulator/car_description/urdf/car.urdf (robot description, URDF)
Before this commit: robot car, 17 links, 16 joints
Joints:
- removed joint board_laster
- added joint board_laser: type fixed, parent board, child laser, origin xyz=0.185 0 0.025 rpy=0 0 3.14159
- joint board_cameraboard: origin xyz=-0.160 0 0.15 -> xyz=-0.025 0 0.15
- joint board_imu: origin xyz=-0.06559 -0.017 0 -> xyz=0.07 -0.017 0
- joint board_marker: origin xyz=0.18 0 0.0025 -> xyz=0.315 0 0.0025
- joint board_support_l: origin xyz=-0.159000 0.053000 0.112000 -> xyz=-0.024000 0.053000 0.112000
- joint board_support_r: origin xyz=-0.159000 -0.053000 0.112000 -> xyz=-0.024000 -0.053000 0.112000
- joint frontwheel_steering_left: origin xyz=0.12 0.08 0.02 -> xyz=0.255 0.08 0.02
- joint frontwheel_steering_right: origin xyz=0.12 -0.08 0.02 -> xyz=0.255 -0.08 0.02
- joint rearwheel_left: origin xyz=-0.135 0.085 0.02 -> xyz=0 0.085 0.02
- joint rearwheel_right: origin xyz=-0.135 -0.085 0.02 -> xyz=0 -0.085 0.02

Commit message: Add bno055 frame

File: catkin_ws/src/autominy_simulator/car_description/urdf/car.urdf (robot description, URDF)
Before this commit: robot car, 17 links, 16 joints
Links:
- added link bno055
Joints:
- added joint joint_board_to_bno055: type fixed, parent board, child bno055, origin xyz=0.235 0.0 0.023 rpy=0 0 1.5708
