Commit message: Improve model

File: catkin_ws/src/autominy_simulator/car_description/urdf/_d435.urdf.xacro (robot description, xacro)
@@ -42,12 +42,11 @@
     </joint>
     <link name="${sensor_name}_link">
-      <visual>
+      <!--<visual>
         <origin xyz="${d435_cam_mount_from_center_offset} ${-d435_cam_depth_py} 0" rpy="${M_PI/2} 0 ${M_PI/2}"/>
         <geometry>
-          <!-- <box size="${d435_cam_width} ${d435_cam_height} ${d435_cam_depth}"/> -->
-          <!--<mesh filename="package://realsense2_camera/meshes/d435/d435.dae" />-->
+          <mesh filename="package://realsense2_camera/meshes/d435/d435.dae" />
         </geometry>
         <material name="${sensor_name}aluminum"/>
-      </visual>
+      </visual>-->
       <collision>
         <origin xyz="0 ${-d435_cam_depth_py} 0" rpy="0 0 0"/>

File: catkin_ws/src/autominy_simulator/car_description/urdf/car.xacro (robot description, xacro)
@@ -2,4 +2,5 @@
 <robot name="car" xmlns:xacro="http://www.ros.org/wiki/xacro">
   <xacro:include filename="$(find car_description)/urdf/_d435.urdf.xacro"/>
+  <xacro:include filename="$(find car_description)/urdf/common.xacro"/>
   <material name="black">
     <color rgba="0.1 0.1 0.1 1"/>
@@ -104,4 +105,24 @@
           <mesh filename="package://car_description/meshes/wheel.dae"/>
         </geometry>
+        <minDepth>0.005</minDepth>
+        <maxContacts>1</maxContacts>
+        <max_contacts>1</max_contacts>
+        <surface>
+          <friction>
+            <ode>
+              <mu>1.0</mu>
+              <mu2>1.0</mu2>
+              <fdir1>0 0 1</fdir1>
+              <slip1>0.0</slip1>
+              <slip2>0.0</slip2>
+            </ode>
+          </friction>
+          <contact>
+            <ode>
+              <min_depth>0.005</min_depth>
+              <kp>1e8</kp>
+            </ode>
+          </contact>
+        </surface>
       </collision>
       <inertial>
@@ -268,5 +289,5 @@
     <parent link="base_link"/>
     <child link="axis_fl"/>
-    <origin xyz="0.255 0.08 0.02"/>
+    <origin xyz="0.255 0.08 0.03"/>
   </joint>
   <joint name="frontwheel_steering_right" type="revolute">
@@ -275,5 +296,5 @@
     <parent link="base_link"/>
     <child link="axis_fr"/>
-    <origin xyz="0.255 -0.08 0.02"/>
+    <origin xyz="0.255 -0.08 0.03"/>
   </joint>
   <joint name="frontwheel_left" type="revolute">
@@ -296,12 +317,12 @@
     <parent link="base_link"/>
     <child link="wheel_bl"/>
-    <origin xyz="0 0.085 0.02"/>
+    <origin xyz="0 0.085 0.03"/>
     <limit effort="0.1" lower="-1000000000000.0" upper="1000000000000.0" velocity="124"/>
-  </joint>
+   </joint>
   <joint name="rearwheel_right" type="revolute">
     <axis xyz="0 1 0"/>
     <parent link="base_link"/>
     <child link="wheel_br"/>
-    <origin xyz="0 -0.085 0.02"/>
+    <origin xyz="0 -0.085 0.03"/>
     <limit effort="0.1" lower="-1000000000000.0" upper="1000000000000.0" velocity="124"/>
   </joint>
