Commit message: Update coordinate systems and include realsense as xacro

File: catkin_ws/src/autominy_simulator/car_description/urdf/car.xacro (robot description, xacro)
@@ -1,4 +1,5 @@
 <?xml version="1.0"?>
-<robot name="car">
+<robot name="car" xmlns:xacro="http://www.ros.org/wiki/xacro">
+  <xacro:include filename="$(find car_robot_model)/urdf/include/_d435.urdf.xacro"/>
   <material name="black">
     <color rgba="0.1 0.1 0.1 1"/>
@@ -33,5 +34,5 @@
   <link name="board">
     <visual>
-      <origin rpy="0.0 0 0" xyz="0.135 0 0"/>
+      <origin rpy="0.0 0 0" xyz="0.115 0 0"/>
       <geometry>
         <mesh filename="package://car_description/meshes/board.dae"/>
@@ -40,5 +41,5 @@
     </visual>
     <collision>
-      <origin rpy="0.0 0 0" xyz="0.135 0 0"/>
+      <origin rpy="0.0 0 0" xyz="0.115 0 0"/>
       <geometry>
         <mesh filename="package://car_description/meshes/board.dae"/>
@@ -46,26 +47,7 @@
     </collision>
     <inertial>
-      <origin rpy="0.0 0 0" xyz="0.135 0 0"/>
+      <origin rpy="0.0 0 0" xyz="0.115 0 0"/>
       <mass value="1.0"/>
       <inertia ixx="0.00213542" ixy="0.0" ixz="0.0" iyy="0.01235417" iyz="0.0" izz="0.01448542"/>
-    </inertial>
-  </link>
-  <link name="camera">
-    <visual>
-      <origin rpy="-2.0944 0 -1.570796" xyz="0 0 0"/>
-      <geometry>
-        <mesh filename="package://car_description/meshes/camera.dae"/>
-      </geometry>
-      <material name="black"/>
-    </visual>
-    <collision>
-      <origin rpy="-2.0944 0 -1.570796" xyz="0 0 0"/>
-      <geometry>
-        <mesh filename="package://car_description/meshes/camera.dae"/>
-      </geometry>
-    </collision>
-    <inertial>
-      <mass value="0.1"/>
-      <inertia ixx="0.00001051" ixy="0.0" ixz="0.0" iyy="0.00006385" iyz="0.0" izz="0.00006403"/>
     </inertial>
   </link>
@@ -90,6 +72,4 @@
     </inertial>
   </link>
-  <link name="camera_bottom_screw_frame"/>
-  <link name="camera_depth_frame"/>
   <link name="laser">
     <visual>
@@ -111,76 +91,28 @@
     </inertial>
   </link>
-  <link name="wheel_fl">
-    <visual>
-      <origin rpy="0.0 0 0" xyz="0 0 0"/>
-      <geometry>
-        <mesh filename="package://car_description/meshes/wheel.dae"/>
-      </geometry>
-      <material name="black"/>
-    </visual>
-    <collision>
-      <geometry>
-        <mesh filename="package://car_description/meshes/wheel.dae"/>
-      </geometry>
-    </collision>
-    <inertial>
-      <mass value="0.05"/>
-      <inertia ixx="0.00001793" ixy="0.0" ixz="0.0" iyy="0.00002867" iyz="0.0" izz="0.00001813"/>
-    </inertial>
-  </link>
-  <link name="wheel_fr">
-    <visual>
-      <origin rpy="0.0 0 0" xyz="0 0 0"/>
-      <geometry>
-        <mesh filename="package://car_description/meshes/wheel.dae"/>
-      </geometry>
-      <material name="black"/>
-    </visual>
-    <collision>
-      <geometry>
-        <mesh filename="package://car_description/meshes/wheel.dae"/>
-      </geometry>
-    </collision>
-    <inertial>
-      <mass value="0.05"/>
-      <inertia ixx="0.00001793" ixy="0.0" ixz="0.0" iyy="0.00002867" iyz="0.0" izz="0.00001813"/>
-    </inertial>
-  </link>
-  <link name="wheel_bl">
-    <visual>
-      <origin rpy="0.0 0 0" xyz="0 0 0"/>
-      <geometry>
-        <mesh filename="package://car_description/meshes/wheel.dae"/>
-      </geometry>
-      <material name="black"/>
-    </visual>
-    <collision>
-      <geometry>
-        <mesh filename="package://car_description/meshes/wheel.dae"/>
-      </geometry>
-    </collision>
-    <inertial>
-      <mass value="0.05"/>
-      <inertia ixx="0.00001793" ixy="0.0" ixz="0.0" iyy="0.00002867" iyz="0.0" izz="0.00001813"/>
-    </inertial>
-  </link>
-  <link name="wheel_br">
-    <visual>
-      <origin rpy="0.0 0 0" xyz="0 0 0"/>
-      <geometry>
-        <mesh filename="package://car_description/meshes/wheel.dae"/>
-      </geometry>
-      <material name="black"/>
-    </visual>
-    <collision>
-      <geometry>>
-        <mesh filename="package://car_description/meshes/wheel.dae"/>
-      </geometry>
-    </collision>
-    <inertial>
-      <mass value="0.05"/>
-      <inertia ixx="0.00001793" ixy="0.0" ixz="0.0" iyy="0.00002867" iyz="0.0" izz="0.00001813"/>
-    </inertial>
-  </link>
+  <xacro:macro name="wheel" params="name">
+    <link name="${name}">
+      <visual>
+        <origin rpy="0.0 0 0" xyz="0 0 0"/>
+        <geometry>
+          <mesh filename="package://car_description/meshes/wheel.dae"/>
+        </geometry>
+        <material name="black"/>
+      </visual>
+      <collision>
+        <geometry>
+          <mesh filename="package://car_description/meshes/wheel.dae"/>
+        </geometry>
+      </collision>
+      <inertial>
+        <mass value="0.05"/>
+        <inertia ixx="0.00001793" ixy="0.0" ixz="0.0" iyy="0.00002867" iyz="0.0" izz="0.00001813"/>
+      </inertial>
+    </link>
+  </xacro:macro>
+  <xacro:wheel name="wheel_fr"/>
+  <xacro:wheel name="wheel_fl"/>
+  <xacro:wheel name="wheel_br"/>
+  <xacro:wheel name="wheel_bl"/>
   <link name="axis_fl">
     <visual>
@@ -293,4 +225,12 @@
   <link name="bno055">
   </link>
+  <!-- front camera -->
+  <xacro:property name="front_camera_name" value="camera"/>
+  <sensor_d435 parent="camera_board" sensor_name="camera">
+    <origin xyz="0.03 0 0.025" rpy="0 0.2 0"/>
+  </sensor_d435>
+  <sensor_d435 parent="camera_board" sensor_name="rear_camera">
+    <origin xyz="-0.02 0 0.025" rpy="0 0.2 3.141"/>
+  </sensor_d435>
   <joint name="joint_board_to_bno055" type="fixed">
       <parent link="board"/>
@@ -301,5 +241,5 @@
     <parent link="base_link"/>
     <child link="board"/>
-    <origin xyz="-0.018 0 0.06"/>
+    <origin xyz="0 0 0.07"/>
   </joint>
   <joint name="board_cameraboard" type="fixed">
@@ -308,19 +248,4 @@
     <origin xyz="-0.025 0 0.15"/>
   </joint>
-  <joint name="camera_cameraboard" type="fixed">
-    <parent link="camera_board"/>
-    <child link="camera"/>
-    <origin xyz="0.035 0 0.03"/>
-  </joint>
-  <joint name="camera_depth" type="fixed">
-    <parent link="camera"/>
-    <child link="camera_depth_frame"/>
-    <origin rpy="-1.57079632679 0 -1.57079632679"/>
-  </joint>
-  <joint name="camera_joint" type="fixed">
-    <origin rpy="0 0 0" xyz="0.035 0 0.03"/>
-    <parent link="camera_board"/>
-    <child link="camera_bottom_screw_frame"/>
-  </joint>
   <joint name="board_laser" type="fixed">
     <parent link="board"/>
@@ -336,5 +261,5 @@
     <parent link="board"/>
     <child link="marker"/>
-    <origin xyz="0.315 0 0.0025"/>
+    <origin xyz="0.30 0 0.0025"/>
   </joint>
   <joint name="frontwheel_steering_left" type="revolute">
@@ -500,5 +425,5 @@
     </plugin>
   </gazebo>
-  <gazebo reference="camera">
+  <gazebo reference="camera_depth_frame">
     <sensor type="depth" name="camera1">
       <always_on>1</always_on>
@@ -506,6 +431,6 @@
       <update_rate>15.0</update_rate>
       <camera>
-        <pose>0 0 0 0 0.30 0</pose>
-        <horizontal_fov>1.59174</horizontal_fov>
+        <pose>0 0 0 0 0.20 0</pose>
+        <horizontal_fov>1.3900031938640904</horizontal_fov>
         <image>
           <width>640</width>
@@ -549,10 +474,10 @@
     </sensor>
   </gazebo>
-  <gazebo reference="camera">
+  <gazebo reference="camera_color_frame">
     <sensor type="camera" name="camera2">
       <update_rate>15.0</update_rate>
       <camera>
-        <pose>0 0 0 0 0.30 0</pose>
-        <horizontal_fov>0.7417649</horizontal_fov>
+        <pose>0 0 0.02 0 0.20 0</pose>
+        <horizontal_fov>0.95417536656506718</horizontal_fov>
         <image>
           <width>640</width>
@@ -576,5 +501,5 @@
         <imageTopicName>image_rect_color</imageTopicName>
         <cameraInfoTopicName>camera_info</cameraInfoTopicName>
-        <frameName>camera</frameName>
+        <frameName>camera_color_optical_frame</frameName>
         <hackBaseline>0.0193</hackBaseline>
         <distortionK1>0.0</distortionK1>

Commit message: Fix car rolling and reset back to normal gravity

File: catkin_ws/src/autominy_simulator/car_description/urdf/car.xacro (robot description, xacro)
@@ -95,5 +95,5 @@
     <link name="${name}">
       <visual>
-        <origin rpy="0.0 0 0" xyz="0 0 0"/>
+        <origin rpy="0 0 0" xyz="0 0 0"/>
         <geometry>
           <mesh filename="package://car_description/meshes/wheel.dae"/>
@@ -102,33 +102,38 @@
       </visual>
       <collision>
+        <origin rpy="0 1.5707 1.5707" xyz="0 0 0"/>
         <geometry>
-          <mesh filename="package://car_description/meshes/wheel.dae"/>
+          <cylinder length="0.025" radius="0.0325" />
         </geometry>
-        <minDepth>0.005</minDepth>
-        <maxContacts>1</maxContacts>
-        <max_contacts>1</max_contacts>
-        <surface>
-          <friction>
-            <ode>
-              <mu>1.0</mu>
-              <mu2>1.0</mu2>
-              <fdir1>0 0 1</fdir1>
-              <slip1>0.0</slip1>
-              <slip2>0.0</slip2>
-            </ode>
-          </friction>
-          <contact>
-            <ode>
-              <min_depth>0.005</min_depth>
-              <kp>1e8</kp>
-            </ode>
-          </contact>
-        </surface>
       </collision>
-      <inertial>
-        <mass value="0.05"/>
-        <inertia ixx="0.00001793" ixy="0.0" ixz="0.0" iyy="0.00002867" iyz="0.0" izz="0.00001813"/>
-      </inertial>
+      <xacro:cylinder_inertial_with_origin radius="0.025" length="0.0325" mass="0.05" >
+        <origin xyz="0 0 0" rpy="0 1.5707 1.5707" />
+      </xacro:cylinder_inertial_with_origin>
     </link>
+    <gazebo reference="${name}">
+      <minDepth>0.005</minDepth>
+      <min_depth>0.005</min_depth>
+      <surface>
+        <friction>
+          <ode>
+            <mu>1.0</mu>
+            <mu2>1.0</mu2>
+            <fdir1>0 0 1</fdir1>
+            <slip1>0.0</slip1>
+            <slip2>0.0</slip2>
+          </ode>
+        </friction>
+        <contact>
+          <ode>
+            <soft_cfm>0.000000001</soft_cfm>
+            <soft_erp>0.2</soft_erp>
+            <kp>1e+10</kp>
+            <kd>10</kd>
+            <max_vel>0.01</max_vel>
+            <min_depth>0.005</min_depth>
+          </ode>
+        </contact>
+      </surface>
+  </gazebo>
   </xacro:macro>
   <xacro:wheel name="wheel_fr"/>

Commit message: Add nuc

File: catkin_ws/src/autominy_simulator/car_description/urdf/car.xacro (robot description, xacro)
@@ -111,29 +111,4 @@
       </xacro:cylinder_inertial_with_origin>
     </link>
-    <gazebo reference="${name}">
-      <minDepth>0.005</minDepth>
-      <min_depth>0.005</min_depth>
-      <surface>
-        <friction>
-          <ode>
-            <mu>1.0</mu>
-            <mu2>1.0</mu2>
-            <fdir1>0 0 1</fdir1>
-            <slip1>0.0</slip1>
-            <slip2>0.0</slip2>
-          </ode>
-        </friction>
-        <contact>
-          <ode>
-            <soft_cfm>0.000000001</soft_cfm>
-            <soft_erp>0.2</soft_erp>
-            <kp>1e+10</kp>
-            <kd>10</kd>
-            <max_vel>0.01</max_vel>
-            <min_depth>0.005</min_depth>
-          </ode>
-        </contact>
-      </surface>
-  </gazebo>
   </xacro:macro>
   <xacro:wheel name="wheel_fr"/>
@@ -250,4 +225,22 @@
   <!-- BNO055 -->
   <link name="bno055">
+  </link>
+  <link name="nuc">
+    <visual>
+      <origin rpy="0 0 0" xyz="0 0 0.022"/>
+      <geometry>
+        <box size="0.11 0.11 0.04" />
+      </geometry>
+      <material name="black"/>
+    </visual>
+    <collision>
+      <origin rpy="0 0 0" xyz="0 0 0.022"/>
+      <geometry>
+        <box size="0.11 0.11 0.04" />
+      </geometry>
+    </collision>
+    <xacro:box_inertial_with_origin x="0.11" y="0.11" z="0.04" mass="0.7" >
+      <origin xyz="0 0 0.025" rpy="0 0 0" />
+    </xacro:box_inertial_with_origin>
   </link>
   <!-- front camera -->
@@ -277,5 +270,5 @@
     <parent link="board"/>
     <child link="laser"/>
-    <origin rpy="0 0 3.14159" xyz="0.185 0 0.025"/>
+    <origin rpy="0 0 3.14159" xyz="0.14 0 0.0625"/>
   </joint>
   <joint name="board_imu" type="fixed">
@@ -288,4 +281,9 @@
     <child link="marker"/>
     <origin xyz="0.30 0 0.0025"/>
+  </joint>
+  <joint name="board_nuc" type="fixed">
+    <parent link="board"/>
+    <child link="nuc"/>
+    <origin xyz="0.16 0 0"/>
   </joint>
   <joint name="frontwheel_steering_left" type="revolute">
@@ -486,5 +484,6 @@
         <pointCloudTopicName>depth/points</pointCloudTopicName>
         <depthImageCameraInfoTopicName>depth/camera_info</depthImageCameraInfoTopicName>
-        <pointCloudCutoff>0.4</pointCloudCutoff>
+        <pointCloudCutoff>0.05</pointCloudCutoff>
+        <pointCloudCutoffMax>15.0</pointCloudCutoffMax>
         <hackBaseline>0.007</hackBaseline>
         <CxPrime>322.3056945800781</CxPrime>
@@ -495,5 +494,5 @@
           <type>gaussian</type>
           <mean>0.0</mean>
-          <stddev>0.01</stddev>
+          <stddev>0.0</stddev>
         </noise>
       </plugin>
@@ -589,3 +588,6 @@
     <material>Gazebo/Black</material>
   </gazebo>
+  <gazebo reference="nuc">
+    <material>Gazebo/Black</material>
+  </gazebo>
 </robot>
