Commit message: Simulation is spawning

File: catkin_ws/src/autominy_simulator/world_description/urdf/circuits/lab.urdf (robot description, URDF)
Before this commit: robot lab, 1 links, 0 joints
Links:
- link base_link: geometry collision mesh filename=file://$(find world_description)/model/world.dae; visual mesh filename=file://$(find world_description)/model/world.dae

File: catkin_ws/src/autominy_simulator/world_description/urdf/roads/road_ground.xacro (robot description, xacro)
@@ -31,5 +31,5 @@
         <origin xyz="0 0 0" rpy="0 0 0"/>
         <geometry>
-          <mesh filename="package://road_description/urdf/roads/dae/${dae}.dae" scale="${size} 1.0 ${size}"/>
+          <mesh filename="file://$(find road_description)/urdf/roads/dae/${dae}.dae" scale="${size} 1.0 ${size}"/>
         </geometry>
       </visual>

File: catkin_ws/src/autominy_simulator/world_description/urdf/roads/road_piece.xacro (robot description, xacro)
@@ -19,5 +19,5 @@
         <origin xyz="0 0 0" rpy="0 0 0"/>
         <geometry>
-          <mesh filename="package://road_description/urdf/roads/dae/${dae}.dae" scale="${size} 1.0 ${size}"/>
+          <mesh filename="file://$(find road_description)/urdf/roads/dae/${dae}.dae" scale="${size} 1.0 ${size}"/>
         </geometry>
       </visual>

File: catkin_ws/src/car_description/urdf/_d435.urdf.xacro (robot description, xacro)
@@ -45,5 +45,5 @@
         <origin xyz="${d435_cam_mount_from_center_offset} ${-d435_cam_depth_py} 0" rpy="${M_PI/2} 0 ${M_PI/2}"/>
         <geometry>
-          <mesh filename="package://realsense2_camera/meshes/d435/d435.dae" />
+          <mesh filename="file://$(find realsense2_camera)/meshes/d435/d435.dae" />
         </geometry>
         <material name="${sensor_name}aluminum"/>

File: catkin_ws/src/car_description/urdf/car.xacro (robot description, xacro)
@@ -25,5 +25,5 @@
       <origin rpy="0.0 0 0" xyz="0.135 0 0.01"/>
       <geometry>
-        <mesh filename="package://car_description/meshes/chasi.dae"/>
+        <mesh filename="file://$(find car_description)/meshes/chasi.dae"/>
       </geometry>
       <material name="black"/>
@@ -32,5 +32,5 @@
       <origin rpy="0.0 0 0" xyz="0.135 0 0.01"/>
       <geometry>
-        <mesh filename="package://car_description/meshes/chasi.dae"/>
+        <mesh filename="file://$(find car_description)/meshes/chasi.dae"/>
       </geometry>
     </collision>
@@ -40,5 +40,5 @@
       <origin rpy="0.0 0 0" xyz="0.115 0 0"/>
       <geometry>
-        <mesh filename="package://car_description/meshes/board.dae"/>
+        <mesh filename="file://$(find car_description)/meshes/board.dae"/>
       </geometry>
       <material name="plastic"/>
@@ -47,5 +47,5 @@
       <origin rpy="0.0 0 0" xyz="0.115 0 0"/>
       <geometry>
-        <mesh filename="package://car_description/meshes/board.dae"/>
+        <mesh filename="file://$(find car_description)/meshes/board.dae"/>
       </geometry>
     </collision>
@@ -60,5 +60,5 @@
       <origin rpy="0.0 0 0" xyz="0 0 0"/>
       <geometry>
-        <mesh filename="package://car_description/meshes/camera_board.dae"/>
+        <mesh filename="file://$(find car_description)/meshes/camera_board.dae"/>
       </geometry>
       <material name="plastic"/>
@@ -67,5 +67,5 @@
       <origin rpy="0.0 0 0" xyz="0 0 0"/>
       <geometry>
-        <mesh filename="package://car_description/meshes/camera_board.dae"/>
+        <mesh filename="file://$(find car_description)/meshes/camera_board.dae"/>
       </geometry>
     </collision>
@@ -81,5 +81,5 @@
         <origin rpy="0 0 0" xyz="0 0 0"/>
         <geometry>
-          <mesh filename="package://car_description/meshes/wheel.dae"/>
+          <mesh filename="file://$(find car_description)/meshes/wheel.dae"/>
         </geometry>
         <material name="black"/>
@@ -157,5 +157,5 @@
     <visual>
       <geometry>
-        <mesh filename="package://car_description/meshes/marker.dae"/>
+        <mesh filename="file://$(find car_description)/meshes/marker.dae"/>
       </geometry>
       <origin rpy="0 0 1.5708" xyz="0 0 0"/>
@@ -262,5 +262,5 @@
     <parent link="$(arg tf_prefix)board"/>
     <child link="$(arg tf_prefix)marker"/>
-    <origin xyz="$(optenv ROS_ESTIMATION_MARKER_X 0.30) $(optenv ROS_ESTIMATION_MARKER_Y 0.0) 0.0025"/>
+    <origin xyz="0.30 0.0 0.0025"/>
   </joint>
   <joint name="$(arg tf_prefix)board_nuc" type="fixed">
@@ -407,8 +407,8 @@
   <gazebo>
     <plugin name="model_car_ground_truth" filename="libgazebo_ros_p3d.so">
-      <frameName>map</frameName>
-      <bodyName>$(arg tf_prefix)base_link</bodyName>
-      <topicName>simulation/odom_ground_truth</topicName>
-      <updateRate>30.0</updateRate>
+      <frame_name>map</frame_name>
+      <body_name>$(arg tf_prefix)base_link</body_name>
+      <topic_name>simulation/odom_ground_truth</topic_name>
+      <update_rate>30.0</update_rate>
     </plugin>
   </gazebo>

File: catkin_ws/src/car_description/urdf/rplidar_a2.xacro (robot description, xacro)
@@ -12,5 +12,5 @@
                 <origin xyz="0 0 0" rpy="0 0 0"/>
                 <geometry>
-                    <mesh filename="package://car_description/meshes/laser.dae"/>
+                    <mesh filename="file://$(find car_description)/meshes/laser.dae"/>
                 </geometry>
             </collision>
@@ -18,7 +18,7 @@
                 <origin xyz="0 0 0" rpy="0 0 0"/>
                 <geometry>
-                    <mesh filename="package://car_description/meshes/laser.dae"/>
+                    <mesh filename="file://$(find car_description)/meshes/laser.dae"/>
                 </geometry>
-                <material name="Black"/>
+                <material name="black"/>
             </visual>
             <inertial>
