Commit message: Use rplidar xacro script

File: catkin_ws/src/car_description/urdf/car.xacro (robot description, xacro)
@@ -2,4 +2,5 @@
 <robot name="car" xmlns:xacro="http://www.ros.org/wiki/xacro">
   <xacro:include filename="$(find car_description)/urdf/_d435.urdf.xacro"/>
+  <xacro:include filename="$(find car_description)/urdf/rplidar_a2.xacro"/>
   <xacro:include filename="$(find car_description)/urdf/common.xacro"/>
   <material name="black">
@@ -71,23 +72,4 @@
       <mass value="0.1"/>
       <inertia ixx="0.00014165" ixy="0.0" ixz="0.0" iyy="0.00006758" iyz="0.0" izz="0.00020865"/>
-    </inertial>
-  </link>
-  <link name="laser">
-    <visual>
-      <origin rpy="0.0 0 0" xyz="0 0 -0.02"/>
-      <geometry>
-        <mesh filename="package://car_description/meshes/laser.dae"/>
-      </geometry>
-      <material name="black"/>
-    </visual>
-    <collision>
-       <origin rpy="0.0 0 0" xyz="0 0 -0.02"/>
-      <geometry>
-        <mesh filename="package://car_description/meshes/laser.dae"/>
-      </geometry>
-    </collision>
-    <inertial>
-      <mass value="0.1"/>
-      <inertia ixx="0.00005965" ixy="0.0" ixz="0.0" iyy="0.00005759" iyz="0.0" izz="0.00009268"/>
     </inertial>
   </link>
@@ -252,4 +234,7 @@
     <origin xyz="-0.02 0 0.025" rpy="0 0.2 3.141"/>
   </sensor_d435>
+  <sensor_rplidar_a2 parent="board" prefix="lidar">
+    <origin xyz="0.14 0 0.0425" rpy="0 0 0"/>
+  </sensor_rplidar_a2>
   <joint name="joint_board_to_bno055" type="fixed">
       <parent link="board"/>
@@ -266,9 +251,4 @@
     <child link="camera_board"/>
     <origin xyz="-0.025 0 0.15"/>
-  </joint>
-  <joint name="board_laser" type="fixed">
-    <parent link="board"/>
-    <child link="laser"/>
-    <origin rpy="0 0 3.14159" xyz="0.14 0 0.0625"/>
   </joint>
   <joint name="board_imu" type="fixed">

Commit message: Fix lidar position and add configurable marker positions

File: catkin_ws/src/car_description/urdf/car.xacro (robot description, xacro)
@@ -260,5 +260,5 @@
     <parent link="board"/>
     <child link="marker"/>
-    <origin xyz="0.30 0 0.0025"/>
+    <origin xyz="$(optenv ROS_ESTIMATION_MARKER_X 0.30) $(optenv ROS_ESTIMATION_MARKER_Y 0.0) 0.0025"/>
   </joint>
   <joint name="board_nuc" type="fixed">

Commit message: Update URDF files so they work on noetic

File: catkin_ws/src/car_description/urdf/car.xacro (robot description, xacro)
@@ -228,13 +228,13 @@
   <!-- front camera -->
   <xacro:property name="front_camera_name" value="camera"/>
-  <sensor_d435 parent="camera_board" sensor_name="camera">
+  <xacro:sensor_d435 parent="camera_board" sensor_name="camera">
     <origin xyz="0.03 0 0.025" rpy="0 0.2 0"/>
-  </sensor_d435>
-  <sensor_d435 parent="camera_board" sensor_name="rear_camera">
+  </xacro:sensor_d435>
+  <xacro:sensor_d435 parent="camera_board" sensor_name="rear_camera">
     <origin xyz="-0.02 0 0.025" rpy="0 0.2 3.141"/>
-  </sensor_d435>
-  <sensor_rplidar_a2 parent="board" prefix="lidar">
+  </xacro:sensor_d435>
+  <xacro:sensor_rplidar_a2 parent="board" prefix="lidar">
     <origin xyz="0.14 0 0.0425" rpy="0 0 0"/>
-  </sensor_rplidar_a2>
+  </xacro:sensor_rplidar_a2>
   <joint name="joint_board_to_bno055" type="fixed">
       <parent link="board"/>

File: catkin_ws/src/car_description/urdf/common.xacro (robot description, xacro)
@@ -2,5 +2,5 @@
 <robot
         xmlns:xacro="http://ros.org/wiki/xacro">
-    <property name="M_PI" value="3.1415926535897931" />
+    <xacro:property name="M_PI" value="3.1415926535897931" />
     <!-- see https://secure.wikimedia.org/wikipedia/en/wiki/List_of_moment_of_inertia_tensors -->
     <!-- #################### versions without origin #################### -->
@@ -36,5 +36,5 @@
         <inertial>
             <mass value="${mass}" />
-            <insert_block name="origin" />
+            <xacro:insert_block name="origin" />
             <inertia ixx="${0.4 * mass * radius * radius}" ixy="0.0" ixz="0.0"
                      iyy="${0.4 * mass * radius * radius}" iyz="0.0"
@@ -45,5 +45,5 @@
         <inertial>
             <mass value="${mass}" />
-            <insert_block name="origin" />
+            <xacro:insert_block name="origin" />
             <inertia ixx="${0.0833333 * mass * (3 * radius * radius + length * length)}" ixy="0.0" ixz="0.0"
                      iyy="${0.0833333 * mass * (3 * radius * radius + length * length)}" iyz="0.0"
@@ -54,5 +54,5 @@
         <inertial>
             <mass value="${mass}" />
-            <insert_block name="origin" />
+            <xacro:insert_block name="origin" />
             <inertia ixx="${0.0833333 * mass * (y*y + z*z)}" ixy="0.0" ixz="0.0"
                      iyy="${0.0833333 * mass * (x*x + z*z)}" iyz="0.0"

Commit message: Make it possible to spawn 2nd car

File: catkin_ws/src/car_description/urdf/car.xacro (robot description, xacro)
@@ -4,4 +4,5 @@
   <xacro:include filename="$(find car_description)/urdf/rplidar_a2.xacro"/>
   <xacro:include filename="$(find car_description)/urdf/common.xacro"/>
+  <xacro:arg name="tf_prefix" default=""/>
   <material name="black">
     <color rgba="0.1 0.1 0.1 1"/>
@@ -19,5 +20,5 @@
     <color rgba="0.95 0.95 0.95 1"/>
   </material>
-  <link name="base_link">
+  <link name="$(arg tf_prefix)base_link">
     <visual>
       <origin rpy="0.0 0 0" xyz="0.135 0 0.01"/>
@@ -34,5 +35,5 @@
     </collision>
   </link>
-  <link name="board">
+  <link name="$(arg tf_prefix)board">
     <visual>
       <origin rpy="0.0 0 0" xyz="0.115 0 0"/>
@@ -54,5 +55,5 @@
     </inertial>
   </link>
-  <link name="camera_board">
+  <link name="$(arg tf_prefix)camera_board">
     <visual>
       <origin rpy="0.0 0 0" xyz="0 0 0"/>
@@ -94,9 +95,9 @@
     </link>
   </xacro:macro>
-  <xacro:wheel name="wheel_fr"/>
-  <xacro:wheel name="wheel_fl"/>
-  <xacro:wheel name="wheel_br"/>
-  <xacro:wheel name="wheel_bl"/>
-  <link name="axis_fl">
+  <xacro:wheel name="$(arg tf_prefix)wheel_fr"/>
+  <xacro:wheel name="$(arg tf_prefix)wheel_fl"/>
+  <xacro:wheel name="$(arg tf_prefix)wheel_br"/>
+  <xacro:wheel name="$(arg tf_prefix)wheel_bl"/>
+  <link name="$(arg tf_prefix)axis_fl">
     <visual>
       <origin rpy="0.0 0 0" xyz="0 0 0"/>
@@ -116,5 +117,5 @@
     </inertial>
   </link>
-  <link name="axis_fr">
+  <link name="$(arg tf_prefix)axis_fr">
     <visual>
       <origin rpy="0.0 0 0" xyz="0 0 0"/>
@@ -134,5 +135,5 @@
     </inertial>
   </link>
-  <link name="imu">
+  <link name="$(arg tf_prefix)imu">
     <visual>
       <geometry>
@@ -152,5 +153,5 @@
     </inertial>
   </link>
-  <link name="marker">
+  <link name="$(arg tf_prefix)marker">
     <visual>
       <geometry>
@@ -169,5 +170,5 @@
     </inertial>
   </link>
-  <link name="support_l">
+  <link name="$(arg tf_prefix)support_l">
     <visual>
       <geometry>
@@ -187,5 +188,5 @@
     </inertial>
   </link>
-  <link name="support_r">
+  <link name="$(arg tf_prefix)support_r">
     <visual>
       <geometry>
@@ -206,7 +207,7 @@
   </link>
   <!-- BNO055 -->
-  <link name="bno055">
-  </link>
-  <link name="nuc">
+  <link name="$(arg tf_prefix)bno055">
+  </link>
+  <link name="$(arg tf_prefix)nuc">
     <visual>
       <origin rpy="0 0 0" xyz="0 0 0.022"/>
@@ -228,41 +229,41 @@
   <!-- front camera -->
   <xacro:property name="front_camera_name" value="camera"/>
-  <xacro:sensor_d435 parent="camera_board" sensor_name="camera">
+  <xacro:sensor_d435 parent="$(arg tf_prefix)camera_board" sensor_name="camera">
     <origin xyz="0.03 0 0.025" rpy="0 0.2 0"/>
   </xacro:sensor_d435>
-  <xacro:sensor_d435 parent="camera_board" sensor_name="rear_camera">
+  <xacro:sensor_d435 parent="$(arg tf_prefix)camera_board" sensor_name="rear_camera">
     <origin xyz="-0.02 0 0.025" rpy="0 0.2 3.141"/>
   </xacro:sensor_d435>
-  <xacro:sensor_rplidar_a2 parent="board" prefix="lidar">
+  <xacro:sensor_rplidar_a2 parent="$(arg tf_prefix)board" prefix="lidar" tf_prefix="$(arg tf_prefix)">
     <origin xyz="0.14 0 0.0425" rpy="0 0 0"/>
   </xacro:sensor_rplidar_a2>
-  <joint name="joint_board_to_bno055" type="fixed">
-      <parent link="board"/>
-      <child link="bno055"/>
+  <joint name="$(arg tf_prefix)joint_board_to_bno055" type="fixed">
+      <parent link="$(arg tf_prefix)board"/>
+      <child link="$(arg tf_prefix)bno055"/>
       <origin xyz="0.235 0.0 0.023" rpy="0 0 1.5708"/>
   </joint>
-  <joint name="base_link_board" type="fixed">
-    <parent link="base_link"/>
-    <child link="board"/>
+  <joint name="$(arg tf_prefix)base_link_board" type="fixed">
+    <parent link="$(arg tf_prefix)base_link"/>
+    <child link="$(arg tf_prefix)board"/>
     <origin xyz="0 0 0.07"/>
   </joint>
-  <joint name="board_cameraboard" type="fixed">
-    <parent link="board"/>
-    <child link="camera_board"/>
+  <joint name="$(arg tf_prefix)board_cameraboard" type="fixed">
+    <parent link="$(arg tf_prefix)board"/>
+    <child link="$(arg tf_prefix)camera_board"/>
     <origin xyz="-0.025 0 0.15"/>
   </joint>
-  <joint name="board_imu" type="fixed">
-    <parent link="board"/>
-    <child link="imu"/>
+  <joint name="$(arg tf_prefix)board_imu" type="fixed">
+    <parent link="$(arg tf_prefix)board"/>
+    <child link="$(arg tf_prefix)imu"/>
     <origin xyz="0.07 -0.017 0"/>
   </joint>
-  <joint name="board_marker" type="fixed">
-    <parent link="board"/>
-    <child link="marker"/>
+  <joint name="$(arg tf_prefix)board_marker" type="fixed">
+    <parent link="$(arg tf_prefix)board"/>
+    <child link="$(arg tf_prefix)marker"/>
     <origin xyz="$(optenv ROS_ESTIMATION_MARKER_X 0.30) $(optenv ROS_ESTIMATION_MARKER_Y 0.0) 0.0025"/>
   </joint>
-  <joint name="board_nuc" type="fixed">
-    <parent link="board"/>
-    <child link="nuc"/>
+  <joint name="$(arg tf_prefix)board_nuc" type="fixed">
+    <parent link="$(arg tf_prefix)board"/>
+    <child link="$(arg tf_prefix)nuc"/>
     <origin xyz="0.16 0 0"/>
   </joint>
@@ -270,6 +271,6 @@
     <axis xyz="0 0 1"/>
     <limit effort="1000.0" lower="-0.55" upper="0.55" velocity="2"/>
-    <parent link="base_link"/>
-    <child link="axis_fl"/>
+    <parent link="$(arg tf_prefix)base_link"/>
+    <child link="$(arg tf_prefix)axis_fl"/>
     <origin xyz="0.255 0.08 0.03"/>
   </joint>
@@ -277,6 +278,6 @@
     <axis xyz="0 0 1"/>
     <limit effort="1000.0" lower="-0.55" upper="0.55" velocity="2"/>
-    <parent link="base_link"/>
-    <child link="axis_fr"/>
+    <parent link="$(arg tf_prefix)base_link"/>
+    <child link="$(arg tf_prefix)axis_fr"/>
     <origin xyz="0.255 -0.08 0.03"/>
   </joint>
@@ -284,53 +285,53 @@
     <axis xyz="0 1 0"/>
     <anchor xyz="0 0 0"/>
-    <parent link="axis_fl"/>
-    <child link="wheel_fl"/>
+    <parent link="$(arg tf_prefix)axis_fl"/>
+    <child link="$(arg tf_prefix)wheel_fl"/>
     <origin xyz="0 0 0"/>
     <limit effort="0.1" lower="-1000000000000.0" upper="1000000000000.0" velocity="124"/>
   </joint>
-  <joint name="frontwheel_right" type="revolute">
+  <joint name="$(arg tf_prefix)frontwheel_right" type="revolute">
     <axis xyz="0 1 0"/>
-    <parent link="axis_fr"/>
-    <child link="wheel_fr"/>
+    <parent link="$(arg tf_prefix)axis_fr"/>
+    <child link="$(arg tf_prefix)wheel_fr"/>
     <origin xyz="0 0 0"/>
     <limit effort="0.1" lower="-1000000000000.0" upper="1000000000000.0" velocity="124"/>
   </joint>
-   <joint name="rearwheel_left" type="revolute">
+   <joint name="$(arg tf_prefix)rearwheel_left" type="revolute">
     <axis xyz="0 1 0"/>
-    <parent link="base_link"/>
-    <child link="wheel_bl"/>
+    <parent link="$(arg tf_prefix)base_link"/>
+    <child link="$(arg tf_prefix)wheel_bl"/>
     <origin xyz="0 0.085 0.03"/>
     <limit effort="0.1" lower="-1000000000000.0" upper="1000000000000.0" velocity="124"/>
    </joint>
-  <joint name="rearwheel_right" type="revolute">
+  <joint name="$(arg tf_prefix)rearwheel_right" type="revolute">
     <axis xyz="0 1 0"/>
-    <parent link="base_link"/>
-    <child link="wheel_br"/>
+    <parent link="$(arg tf_prefix)base_link"/>
+    <child link="$(arg tf_prefix)wheel_br"/>
     <origin xyz="0 -0.085 0.03"/>
     <limit effort="0.1" lower="-1000000000000.0" upper="1000000000000.0" velocity="124"/>
   </joint>
-  <joint name="board_support_l" type="fixed">
-    <parent link="board"/>
-    <child link="support_l"/>
+  <joint name="$(arg tf_prefix)board_support_l" type="fixed">
+    <parent link="$(arg tf_prefix)board"/>
+    <child link="$(arg tf_prefix)support_l"/>
     <origin xyz="-0.024000 0.053000 0.112000"/>
   </joint>
-  <joint name="board_support_r" type="fixed">
-    <parent link="board"/>
-    <child link="support_r"/>
+  <joint name="$(arg tf_prefix)board_support_r" type="fixed">
+    <parent link="$(arg tf_prefix)board"/>
+    <child link="$(arg tf_prefix)support_r"/>
     <origin xyz="-0.024000 -0.053000 0.112000"/>
   </joint>
-  <transmission name="steering_front_left_wheel">
+  <transmission name="$(arg tf_prefix)steering_front_left_wheel">
     <type>transmission_interface/SimpleTransmission</type>
-    <joint name="frontwheel_steering_left">
+    <joint name="$(arg tf_prefix)frontwheel_steering_left">
       <hardwareInterface>hardware_interface/EffortJointInterface</hardwareInterface>
     </joint>
-    <actuator name="front_left_steering_motor">
+    <actuator name="$(arg tf_prefix)front_left_steering_motor">
       <hardwareInterface>hardware_interface/EffortJointInterface</hardwareInterface>
       <mechanicalReduction>1</mechanicalReduction>
     </actuator>
   </transmission>
-  <transmission name="steering_front_right_wheel">
+  <transmission name="$(arg tf_prefix)steering_front_right_wheel">
     <type>transmission_interface/SimpleTransmission</type>
-    <joint name="frontwheel_steering_right">
+    <joint name="$(arg tf_prefix)frontwheel_steering_right">
       <hardwareInterface>hardware_interface/EffortJointInterface</hardwareInterface>
     </joint>
@@ -340,60 +341,60 @@
     </actuator>
   </transmission>
-  <transmission name="tran_front_left_wheel">
+  <transmission name="$(arg tf_prefix)tran_front_left_wheel">
     <type>transmission_interface/SimpleTransmission</type>
-    <joint name="frontwheel_left">
+    <joint name="$(arg tf_prefix)frontwheel_left">
       <hardwareInterface>hardware_interface/EffortJointInterface</hardwareInterface>
     </joint>
-    <actuator name="front_left_wheel_motor">
+    <actuator name="$(arg tf_prefix)front_left_wheel_motor">
       <hardwareInterface>hardware_interface/EffortJointInterface</hardwareInterface>
       <mechanicalReduction>1</mechanicalReduction>
     </actuator>
   </transmission>
-  <transmission name="tran_front_right_wheel">
+  <transmission name="$(arg tf_prefix)tran_front_right_wheel">
     <type>transmission_interface/SimpleTransmission</type>
-    <joint name="frontwheel_right">
+    <joint name="$(arg tf_prefix)frontwheel_right">
       <hardwareInterface>hardware_interface/EffortJointInterface</hardwareInterface>
     </joint>
-    <actuator name="front_right_wheel_motor">
+    <actuator name="$(arg tf_prefix)front_right_wheel_motor">
       <hardwareInterface>hardware_interface/EffortJointInterface</hardwareInterface>
       <mechanicalReduction>1</mechanicalReduction>
     </actuator>
   </transmission>
-  <transmission name="tran_rear_left">
+  <transmission name="$(arg tf_prefix)tran_rear_left">
     <type>transmission_interface/SimpleTransmission</type>
-    <joint name="rearwheel_left">
+    <joint name="$(arg tf_prefix)rearwheel_left">
       <hardwareInterface>hardware_interface/EffortJointInterface</hardwareInterface>
     </joint>
-    <actuator name="rear_left_motor">
+    <actuator name="$(arg tf_prefix)rear_left_motor">
       <hardwareInterface>hardware_interface/EffortJointInterface</hardwareInterface>
       <mechanicalReduction>1</mechanicalReduction>
     </actuator>
   </transmission>
-  <transmission name="tran_rear_right">
+  <transmission name="$(arg tf_prefix)tran_rear_right">
     <type>transmission_interface/SimpleTransmission</type>
-    <joint name="rearwheel_right">
+    <joint name="$(arg tf_prefix)rearwheel_right">
       <hardwareInterface>hardware_interface/EffortJointInterface</hardwareInterface>
     </joint>
-    <actuator name="rear_right_motor">
+    <actuator name="$(arg tf_prefix)rear_right_motor">
       <hardwareInterface>hardware_interface/EffortJointInterface</hardwareInterface>
       <mechanicalReduction>1</mechanicalReduction>
     </actuator>
   </transmission>
-  <gazebo reference="rearwheel_left">
+  <gazebo reference="$(arg tf_prefix)rearwheel_left">
     <implicitSpringDamper>true</implicitSpringDamper>
   </gazebo>
-  <gazebo reference="rearwheel_right">
+  <gazebo reference="$(arg tf_prefix)rearwheel_right">
     <implicitSpringDamper>true</implicitSpringDamper>
   </gazebo>
-  <gazebo reference="frontwheel_right">
+  <gazebo reference="$(arg tf_prefix)frontwheel_right">
     <implicitSpringDamper>true</implicitSpringDamper>
   </gazebo>
-  <gazebo reference="frontwheel_left">
+  <gazebo reference="$(arg tf_prefix)frontwheel_left">
     <implicitSpringDamper>true</implicitSpringDamper>
   </gazebo>
-  <gazebo reference="frontwheel_steering_right">
+  <gazebo reference="$(arg tf_prefix)frontwheel_steering_right">
     <implicitSpringDamper>true</implicitSpringDamper>
   </gazebo>
-  <gazebo reference="frontwheel_steering_left">
+  <gazebo reference="$(arg tf_prefix)frontwheel_steering_left">
     <implicitSpringDamper>true</implicitSpringDamper>
   </gazebo>
@@ -406,6 +407,6 @@
     <plugin name="model_car_ground_truth" filename="libgazebo_ros_p3d.so">
       <frameName>map</frameName>
-      <bodyName>base_link</bodyName>
-      <topicName>/simulation/odom_ground_truth</topicName>
+      <bodyName>$(arg tf_prefix)base_link</bodyName>
+      <topicName>simulation/odom_ground_truth</topicName>
       <updateRate>30.0</updateRate>
     </plugin>
@@ -416,5 +417,5 @@
       <robotNamespace>/</robotNamespace>
       <bodyName>imu</bodyName>
-      <frameId>imu</frameId>
+      <frameId>$(arg tf_prefix)imu</frameId>
       <topicName>sensors/imu</topicName>
       <accelOffset>0 0 0</accelOffset>
@@ -429,5 +430,5 @@
     </plugin>
   </gazebo>
-  <gazebo reference="camera_depth_frame">
+  <gazebo reference="$(arg tf_prefix)camera_depth_frame">
     <sensor type="depth" name="camera1">
       <always_on>1</always_on>
@@ -458,5 +459,5 @@
         <updateRate>15.0</updateRate>
         <cameraName>sensors/camera</cameraName>
-        <frameName>camera_depth_optical_frame</frameName>
+        <frameName>$(arg tf_prefix)camera_depth_optical_frame</frameName>
         <imageTopicName>infra1/image_rect_raw</imageTopicName>
         <cameraInfoTopicName>infra1/camera_info</cameraInfoTopicName>
@@ -479,5 +480,5 @@
     </sensor>
   </gazebo>
-  <gazebo reference="camera_color_frame">
+  <gazebo reference="$(arg tf_prefix)camera_color_frame">
     <sensor type="camera" name="camera2">
       <update_rate>15.0</update_rate>
@@ -506,5 +507,5 @@
         <imageTopicName>image_rect_color</imageTopicName>
         <cameraInfoTopicName>camera_info</cameraInfoTopicName>
-        <frameName>camera_color_optical_frame</frameName>
+        <frameName>$(arg tf_prefix)camera_color_optical_frame</frameName>
         <hackBaseline>0.0193</hackBaseline>
         <distortionK1>0.0</distortionK1>
@@ -516,5 +517,5 @@
     </sensor>
   </gazebo>
-  <gazebo reference="laser">
+  <gazebo reference="$(arg tf_prefix)laser">
     <sensor type="ray" name="rp_lidar_sensor">
       <pose>0 0 0 0 0 0</pose>
@@ -541,32 +542,32 @@
       </ray>
       <plugin name="gazebo_ros_head_hokuyo_controller" filename="libgazebo_ros_laser.so">
-        <topicName>/sensors/rplidar/scan</topicName>
-        <frameName>laser</frameName>
+        <topicName>sensors/rplidar/scan</topicName>
+        <frameName>$(arg tf_prefix)laser</frameName>
       </plugin>
     </sensor>
   </gazebo>
-  <gazebo reference="wheel_fl">
+  <gazebo reference="$(arg tf_prefix)wheel_fl">
     <mu1>1.34</mu1>
     <mu2>1.34</mu2>
   </gazebo>
-  <gazebo reference="wheel_fr">
+  <gazebo reference="$(arg tf_prefix)wheel_fr">
     <mu1>1.34</mu1>
     <mu2>1.34</mu2>
   </gazebo>
-  <gazebo reference="wheel_br">
+  <gazebo reference="$(arg tf_prefix)wheel_br">
     <mu1>1.34</mu1>
     <mu2>1.34</mu2>
   </gazebo>
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
File: catkin_ws/src/car_description/urdf/rplidar_a2.xacro (robot description, xacro)
@@ -2,11 +2,11 @@
 <robot xmlns:xacro="http://www.ros.org/wiki/xacro">
     <xacro:macro name="sensor_rplidar_a2"
-                 params="prefix parent prefix_topic:='front_laser' *origin min_angle:=-3.14159 max_angle:=3.14159">
-        <joint name="${prefix}_base_joint" type="fixed">
+                 params="prefix parent tf_prefix prefix_topic:='front_laser' *origin min_angle:=-3.14159 max_angle:=3.14159">
+        <joint name="${tf_prefix}${prefix}_base_joint" type="fixed">
             <xacro:insert_block name="origin"/>
             <parent link="${parent}"/>
-            <child link="${prefix}_base_link"/>
+            <child link="${tf_prefix}${prefix}_base_link"/>
         </joint>
-        <link name="${prefix}_base_link">
+        <link name="${tf_prefix}${prefix}_base_link">
             <collision>
                 <origin xyz="0 0 0" rpy="0 0 0"/>
@@ -28,10 +28,10 @@
             </inertial>
         </link>
-        <joint name="${prefix}_laser_joint" type="fixed">
+        <joint name="${tf_prefix}${prefix}_laser_joint" type="fixed">
             <origin xyz="0 0 0.03086" rpy="0 0 3.1415"/>
-            <parent link="${prefix}_base_link"/>
-            <child link="laser"/>
+            <parent link="${tf_prefix}${prefix}_base_link"/>
+            <child link="${tf_prefix}laser"/>
         </joint>
-        <link name="laser">
+        <link name="${tf_prefix}laser">
         </link>
     </xacro:macro>
