Commit message: Fix some more frames

File: catkin_ws/src/car_description/urdf/car.xacro (robot description, xacro)
@@ -1,4 +1,4 @@
 <?xml version="1.0"?>
-<robot name="car" xmlns:xacro="http://www.ros.org/wiki/xacro">
+<robot name="$(arg car_name)" xmlns:xacro="http://www.ros.org/wiki/xacro">
   <xacro:include filename="$(find car_description)/urdf/_d435.urdf.xacro"/>
   <xacro:include filename="$(find car_description)/urdf/rplidar_a2.xacro"/>
@@ -268,5 +268,5 @@
     <origin xyz="0.16 0 0"/>
   </joint>
-  <joint name="frontwheel_steering_left" type="revolute">
+  <joint name="$(arg tf_prefix)frontwheel_steering_left" type="revolute">
     <axis xyz="0 0 1"/>
     <limit effort="1000.0" lower="-0.55" upper="0.55" velocity="2"/>
@@ -275,5 +275,5 @@
     <origin xyz="0.255 0.08 0.03"/>
   </joint>
-  <joint name="frontwheel_steering_right" type="revolute">
+  <joint name="$(arg tf_prefix)frontwheel_steering_right" type="revolute">
     <axis xyz="0 0 1"/>
     <limit effort="1000.0" lower="-0.55" upper="0.55" velocity="2"/>
@@ -282,5 +282,5 @@
     <origin xyz="0.255 -0.08 0.03"/>
   </joint>
-  <joint name="frontwheel_left" type="revolute">
+  <joint name="$(arg tf_prefix)frontwheel_left" type="revolute">
     <axis xyz="0 1 0"/>
     <anchor xyz="0 0 0"/>
@@ -401,5 +401,5 @@
   <gazebo>
     <plugin filename="libgazebo_ros_control.so" name="gazebo_ros_control">
-      <robotNamespace>model_car</robotNamespace>
+      <robotNamespace>$(arg car_name)</robotNamespace>
     </plugin>
   </gazebo>

Commit message: Good progress on simulation

File: catkin_ws/src/car_description/urdf/car.xacro (robot description, xacro)
@@ -79,5 +79,5 @@
     <link name="${name}">
       <visual>
-        <origin rpy="0 0 0" xyz="0 0 0"/>
+        <origin rpy="0.0 0.0 0.0" xyz="0.0 0.0 0.0"/>
         <geometry>
           <mesh filename="file://$(find car_description)/meshes/wheel.dae"/>
@@ -102,5 +102,5 @@
   <link name="$(arg tf_prefix)axis_fl">
     <visual>
-      <origin rpy="0.0 0 0" xyz="0 0 0"/>
+      <origin rpy="0.0 0.0 0.0" xyz="0.0 0.0 0.0"/>
       <geometry>
         <box size="0.001 0.001 0.001"/>
@@ -120,5 +120,5 @@
   <link name="$(arg tf_prefix)axis_fr">
     <visual>
-      <origin rpy="0.0 0 0" xyz="0 0 0"/>
+      <origin rpy="0.0 0.0 0.0" xyz="0.0 0.0 0.0"/>
       <geometry>
         <box size="0.001 0.001 0.001"/>
@@ -274,5 +274,5 @@
     <parent link="$(arg tf_prefix)base_link"/>
     <child link="$(arg tf_prefix)axis_fl"/>
-    <origin xyz="0.255 0.08 0.03"/>
+    <origin xyz="0.255 0.08 0.03" rpy="0.0 0.0 0.0"/>
   </joint>
   <joint name="$(arg tf_prefix)frontwheel_steering_right" type="revolute">
@@ -281,12 +281,11 @@
     <parent link="$(arg tf_prefix)base_link"/>
     <child link="$(arg tf_prefix)axis_fr"/>
-    <origin xyz="0.255 -0.08 0.03"/>
+    <origin xyz="0.255 -0.08 0.03" rpy="0.0 0.0 0.0" />
   </joint>
   <joint name="$(arg tf_prefix)frontwheel_left" type="revolute">
     <axis xyz="0 1 0"/>
-    <anchor xyz="0 0 0"/>
     <parent link="$(arg tf_prefix)axis_fl"/>
     <child link="$(arg tf_prefix)wheel_fl"/>
-    <origin xyz="0 0 0"/>
+    <origin xyz="0 0 0" rpy="0.0 0.0 0.0"/>
     <limit effort="0.1" lower="-1000000000000.0" upper="1000000000000.0" velocity="124"/>
   </joint>
@@ -295,5 +294,5 @@
     <parent link="$(arg tf_prefix)axis_fr"/>
     <child link="$(arg tf_prefix)wheel_fr"/>
-    <origin xyz="0 0 0"/>
+    <origin xyz="0 0 0" rpy="0.0 0.0 0.0"/>
     <limit effort="0.1" lower="-1000000000000.0" upper="1000000000000.0" velocity="124"/>
   </joint>
@@ -302,5 +301,5 @@
     <parent link="$(arg tf_prefix)base_link"/>
     <child link="$(arg tf_prefix)wheel_bl"/>
-    <origin xyz="0 0.085 0.03"/>
+    <origin xyz="0 0.085 0.03" rpy="0.0 0.0 0.0"/>
     <limit effort="0.1" lower="-1000000000000.0" upper="1000000000000.0" velocity="124"/>
    </joint>
@@ -309,5 +308,5 @@
     <parent link="$(arg tf_prefix)base_link"/>
     <child link="$(arg tf_prefix)wheel_br"/>
-    <origin xyz="0 -0.085 0.03"/>
+    <origin xyz="0 -0.085 0.03" rpy="0.0 0.0 0.0" />
     <limit effort="0.1" lower="-1000000000000.0" upper="1000000000000.0" velocity="124"/>
   </joint>
@@ -322,64 +321,42 @@
     <origin xyz="-0.024000 -0.053000 0.112000"/>
   </joint>
-  <transmission name="$(arg tf_prefix)steering_front_left_wheel">
-    <type>transmission_interface/SimpleTransmission</type>
-    <joint name="$(arg tf_prefix)frontwheel_steering_left">
-      <hardwareInterface>hardware_interface/EffortJointInterface</hardwareInterface>
-    </joint>
-    <actuator name="$(arg tf_prefix)front_left_steering_motor">
-      <hardwareInterface>hardware_interface/EffortJointInterface</hardwareInterface>
-      <mechanicalReduction>1</mechanicalReduction>
-    </actuator>
-  </transmission>
-  <transmission name="$(arg tf_prefix)steering_front_right_wheel">
-    <type>transmission_interface/SimpleTransmission</type>
-    <joint name="$(arg tf_prefix)frontwheel_steering_right">
-      <hardwareInterface>hardware_interface/EffortJointInterface</hardwareInterface>
-    </joint>
-    <actuator name="front_right_steering_motor">
-      <hardwareInterface>hardware_interface/EffortJointInterface</hardwareInterface>
-      <mechanicalReduction>1</mechanicalReduction>
-    </actuator>
-  </transmission>
-  <transmission name="$(arg tf_prefix)tran_front_left_wheel">
-    <type>transmission_interface/SimpleTransmission</type>
-    <joint name="$(arg tf_prefix)frontwheel_left">
-      <hardwareInterface>hardware_interface/EffortJointInterface</hardwareInterface>
-    </joint>
-    <actuator name="$(arg tf_prefix)front_left_wheel_motor">
-      <hardwareInterface>hardware_interface/EffortJointInterface</hardwareInterface>
-      <mechanicalReduction>1</mechanicalReduction>
-    </actuator>
-  </transmission>
-  <transmission name="$(arg tf_prefix)tran_front_right_wheel">
-    <type>transmission_interface/SimpleTransmission</type>
-    <joint name="$(arg tf_prefix)frontwheel_right">
-      <hardwareInterface>hardware_interface/EffortJointInterface</hardwareInterface>
-    </joint>
-    <actuator name="$(arg tf_prefix)front_right_wheel_motor">
-      <hardwareInterface>hardware_interface/EffortJointInterface</hardwareInterface>
-      <mechanicalReduction>1</mechanicalReduction>
-    </actuator>
-  </transmission>
-  <transmission name="$(arg tf_prefix)tran_rear_left">
-    <type>transmission_interface/SimpleTransmission</type>
-    <joint name="$(arg tf_prefix)rearwheel_left">
-      <hardwareInterface>hardware_interface/EffortJointInterface</hardwareInterface>
-    </joint>
-    <actuator name="$(arg tf_prefix)rear_left_motor">
-      <hardwareInterface>hardware_interface/EffortJointInterface</hardwareInterface>
-      <mechanicalReduction>1</mechanicalReduction>
-    </actuator>
-  </transmission>
-  <transmission name="$(arg tf_prefix)tran_rear_right">
-    <type>transmission_interface/SimpleTransmission</type>
-    <joint name="$(arg tf_prefix)rearwheel_right">
-      <hardwareInterface>hardware_interface/EffortJointInterface</hardwareInterface>
-    </joint>
-    <actuator name="$(arg tf_prefix)rear_right_motor">
-      <hardwareInterface>hardware_interface/EffortJointInterface</hardwareInterface>
-      <mechanicalReduction>1</mechanicalReduction>
-    </actuator>
-  </transmission>
+    <ros2_control name="GazeboSystem" type="system">
+        <hardware>
+            <plugin>gazebo_ros2_control/GazeboSystem</plugin>
+        </hardware>
+        <joint name="$(arg tf_prefix)rearwheel_left">
+            <command_interface name="effort" />
+          <state_interface name="position"/>
+          <state_interface name="velocity"/>
+        </joint>
+        <joint name="$(arg tf_prefix)rearwheel_right">
+          <command_interface name="effort">
+          </command_interface>
+          <state_interface name="position"/>
+          <state_interface name="velocity"/>
+        </joint>
+        <joint name="$(arg tf_prefix)frontwheel_left">
+        <command_interface name="effort"/>
+          <state_interface name="position"/>
+          <state_interface name="velocity"/>
+        </joint>
+        <joint name="$(arg tf_prefix)frontwheel_right">
+          <command_interface name="effort">
+          </command_interface>
+          <state_interface name="position"/>
+          <state_interface name="velocity"/>
+        </joint>
+        <joint name="$(arg tf_prefix)frontwheel_steering_left">
+        <command_interface name="effort"/>
+            <state_interface name="position"/>
+            <state_interface name="velocity"/>
+        </joint>
+        <joint name="$(arg tf_prefix)frontwheel_steering_right">
+          <command_interface name="effort">
+          </command_interface>
+          <state_interface name="position"/>
+          <state_interface name="velocity"/>
+        </joint>
+    </ros2_control>
   <gazebo reference="$(arg tf_prefix)rearwheel_left">
     <implicitSpringDamper>true</implicitSpringDamper>
@@ -400,9 +377,9 @@
     <implicitSpringDamper>true</implicitSpringDamper>
   </gazebo>
-  <gazebo>
-    <plugin filename="libgazebo_ros_control.so" name="gazebo_ros_control">
-      <robotNamespace>$(arg agent_prefix)/model_car</robotNamespace>
-    </plugin>
-  </gazebo>
+    <gazebo>
+      <plugin filename="libgazebo_ros2_control.so" name="gazebo_ros2_control">
+        <parameters>$(find sim_car_controller)/config/control.yaml</parameters>
+      </plugin>
+    </gazebo>
   <gazebo>
     <plugin name="model_car_ground_truth" filename="libgazebo_ros_p3d.so">

Commit message: Fix model stability
HACK: The CoM is below the ground now

File: catkin_ws/src/car_description/urdf/car.xacro (robot description, xacro)
@@ -35,4 +35,7 @@
       </geometry>
     </collision>
+    <xacro:box_inertial_with_origin mass="30.0" x="0.2" y="0.1" z="0.05">
+      <origin rpy="0.0 0 0" xyz="0.115 0 -0.1" />
+    </xacro:box_inertial_with_origin>
   </link>
   <link name="$(arg tf_prefix)board">
@@ -50,9 +53,7 @@
       </geometry>
     </collision>
-    <inertial>
-      <origin rpy="0.0 0 0" xyz="0.115 0 0"/>
-      <mass value="1.0"/>
-      <inertia ixx="0.00213542" ixy="0.0" ixz="0.0" iyy="0.01235417" iyz="0.0" izz="0.01448542"/>
-    </inertial>
+    <xacro:box_inertial_with_origin x="0.3" y="0.1" z="0.1" mass="0.3" >
+      <origin xyz="0 0 0" rpy="0 0 0" />
+    </xacro:box_inertial_with_origin>
   </link>
   <link name="$(arg tf_prefix)camera_board">
@@ -91,8 +92,14 @@
         </geometry>
       </collision>
-      <xacro:cylinder_inertial_with_origin radius="0.025" length="0.0325" mass="0.05" >
+      <xacro:cylinder_inertial_with_origin radius="0.025" length="0.0325" mass="0.1" >
         <origin xyz="0 0 0" rpy="0 1.5707 1.5707" />
       </xacro:cylinder_inertial_with_origin>
     </link>
+    <gazebo reference="${name}">
+      <mu1>1.23</mu1>
+      <mu2>1.23</mu2>
+      <kp>1000000.0</kp> <!--contact stiffness-->
+      <kd>100.0</kd> <!--damping-->
+    </gazebo>
   </xacro:macro>
   <xacro:wheel name="$(arg tf_prefix)wheel_fr"/>
@@ -113,8 +120,5 @@
       </geometry>
     </collision>
-    <inertial>
-      <mass value="0.1"/>
-      <inertia ixx="0.00000002" ixy="0.0" ixz="0.0" iyy="0.00000002" iyz="0.0" izz="0.00000002"/>
-    </inertial>
+    <xacro:sphere_inertial radius="0.02" mass="0.1" />
   </link>
   <link name="$(arg tf_prefix)axis_fr">
@@ -131,8 +135,5 @@
       </geometry>
     </collision>
-    <inertial>
-      <mass value="0.1"/>
-      <inertia ixx="0.00000002" ixy="0.0" ixz="0.0" iyy="0.00000002" iyz="0.0" izz="0.00000002"/>
-    </inertial>
+    <xacro:sphere_inertial radius="0.02" mass="0.1" />
   </link>
   <link name="$(arg tf_prefix)imu">
@@ -271,43 +272,49 @@
   <joint name="$(arg tf_prefix)frontwheel_steering_left" type="revolute">
     <axis xyz="0 0 1"/>
-    <limit effort="1000.0" lower="-0.55" upper="0.55" velocity="2"/>
+    <limit effort="0.001" lower="-0.60" upper="0.60" velocity="1.0"/>
     <parent link="$(arg tf_prefix)base_link"/>
     <child link="$(arg tf_prefix)axis_fl"/>
     <origin xyz="0.255 0.08 0.03" rpy="0.0 0.0 0.0"/>
+    <dynamics damping="0.1" friction="0.01"/>
   </joint>
   <joint name="$(arg tf_prefix)frontwheel_steering_right" type="revolute">
     <axis xyz="0 0 1"/>
-    <limit effort="1000.0" lower="-0.55" upper="0.55" velocity="2"/>
+    <limit effort="0.001" lower="-0.60" upper="0.60" velocity="1.0"/>
     <parent link="$(arg tf_prefix)base_link"/>
     <child link="$(arg tf_prefix)axis_fr"/>
     <origin xyz="0.255 -0.08 0.03" rpy="0.0 0.0 0.0" />
-  </joint>
-  <joint name="$(arg tf_prefix)frontwheel_left" type="revolute">
+    <dynamics damping="0.1" friction="0.01"/>
+  </joint>
+  <joint name="$(arg tf_prefix)frontwheel_left" type="continuous">
     <axis xyz="0 1 0"/>
     <parent link="$(arg tf_prefix)axis_fl"/>
     <child link="$(arg tf_prefix)wheel_fl"/>
     <origin xyz="0 0 0" rpy="0.0 0.0 0.0"/>
-    <limit effort="0.1" lower="-1000000000000.0" upper="1000000000000.0" velocity="124"/>
-  </joint>
-  <joint name="$(arg tf_prefix)frontwheel_right" type="revolute">
+    <limit effort="100.0" velocity="100.0"/>
+    <dynamics damping="0.1" friction="0.01"/>
+  </joint>
+  <joint name="$(arg tf_prefix)frontwheel_right" type="continuous">
     <axis xyz="0 1 0"/>
     <parent link="$(arg tf_prefix)axis_fr"/>
     <child link="$(arg tf_prefix)wheel_fr"/>
     <origin xyz="0 0 0" rpy="0.0 0.0 0.0"/>
-    <limit effort="0.1" lower="-1000000000000.0" upper="1000000000000.0" velocity="124"/>
-  </joint>
-   <joint name="$(arg tf_prefix)rearwheel_left" type="revolute">
+    <limit effort="100.0" velocity="100.0"/>
+    <dynamics damping="0.1" friction="0.01"/>
+  </joint>
+   <joint name="$(arg tf_prefix)rearwheel_left" type="continuous">
     <axis xyz="0 1 0"/>
     <parent link="$(arg tf_prefix)base_link"/>
     <child link="$(arg tf_prefix)wheel_bl"/>
     <origin xyz="0 0.085 0.03" rpy="0.0 0.0 0.0"/>
-    <limit effort="0.1" lower="-1000000000000.0" upper="1000000000000.0" velocity="124"/>
+    <limit effort="100.0" velocity="100.0"/>
+     <dynamics damping="0.1" friction="0.01"/>
    </joint>
-  <joint name="$(arg tf_prefix)rearwheel_right" type="revolute">
+  <joint name="$(arg tf_prefix)rearwheel_right" type="continuous">
     <axis xyz="0 1 0"/>
     <parent link="$(arg tf_prefix)base_link"/>
     <child link="$(arg tf_prefix)wheel_br"/>
     <origin xyz="0 -0.085 0.03" rpy="0.0 0.0 0.0" />
-    <limit effort="0.1" lower="-1000000000000.0" upper="1000000000000.0" velocity="124"/>
+    <limit effort="100.0" velocity="100.0"/>
+    <dynamics damping="0.1" friction="0.01"/>
   </joint>
   <joint name="$(arg tf_prefix)board_support_l" type="fixed">
@@ -347,6 +354,6 @@
         <joint name="$(arg tf_prefix)frontwheel_steering_left">
           <command_interface name="position">
-            <param name="min">-1</param>
-            <param name="max">1</param>
+            <param name="min">-0.60</param>
+            <param name="max">0.60</param>
           </command_interface>
           <state_interface name="position" />
@@ -355,6 +362,6 @@
         <joint name="$(arg tf_prefix)frontwheel_steering_right">
           <command_interface name="position">
-            <param name="min">-1</param>
-            <param name="max">1</param>
+            <param name="min">-0.60</param>
+            <param name="max">0.60</param>
           </command_interface>
           <state_interface name="position" />
@@ -589,20 +596,4 @@
     </sensor>
   </gazebo>
-  <gazebo reference="$(arg tf_prefix)wheel_fl">
-    <mu1>1.34</mu1>
-    <mu2>1.34</mu2>
-  </gazebo>
-  <gazebo reference="$(arg tf_prefix)wheel_fr">
-    <mu1>1.34</mu1>
-    <mu2>1.34</mu2>
-  </gazebo>
-  <gazebo reference="$(arg tf_prefix)wheel_br">
-    <mu1>1.34</mu1>
-    <mu2>1.34</mu2>
-  </gazebo>
-  <gazebo reference="$(arg tf_prefix)wheel_bl">
-    <mu1>1.34</mu1>
-    <mu2>1.34</mu2>
-  </gazebo>
   <gazebo reference="$(arg tf_prefix)support_r">
     <material>Gazebo/Black</material>

Commit message: PD controller to simulate motor inertia

File: catkin_ws/src/car_description/urdf/car.xacro (robot description, xacro)
@@ -36,5 +36,5 @@
     </collision>
     <xacro:box_inertial_with_origin mass="30.0" x="0.2" y="0.1" z="0.05">
-      <origin rpy="0.0 0 0" xyz="0.115 0 -0.1" />
+      <origin rpy="0.0 0 0" xyz="0.115 0 0.0" />
     </xacro:box_inertial_with_origin>
   </link>
@@ -97,8 +97,9 @@
     </link>
     <gazebo reference="${name}">
-      <mu1>1.23</mu1>
-      <mu2>1.23</mu2>
+      <mu1>0.9</mu1>
+      <mu2>0.9</mu2>
       <kp>1000000.0</kp> <!--contact stiffness-->
-      <kd>100.0</kd> <!--damping-->
+      <kd>1.0</kd> <!--damping-->
+      <minDepth>0.001</minDepth>
     </gazebo>
   </xacro:macro>
@@ -117,23 +118,23 @@
     <collision>
       <geometry>
+        <box size="0 0 0"/>
+      </geometry>
+    </collision>
+    <xacro:sphere_inertial radius="0.02" mass="0.15" />
+  </link>
+  <link name="$(arg tf_prefix)axis_fr">
+    <visual>
+      <origin rpy="0.0 0.0 0.0" xyz="0.0 0.0 0.0"/>
+      <geometry>
+        <box size="0 0 0"/>
+      </geometry>
+      <material name="black"/>
+    </visual>
+    <collision>
+      <geometry>
         <box size="0.001 0.001 0.001"/>
       </geometry>
     </collision>
-    <xacro:sphere_inertial radius="0.02" mass="0.1" />
-  </link>
-  <link name="$(arg tf_prefix)axis_fr">
-    <visual>
-      <origin rpy="0.0 0.0 0.0" xyz="0.0 0.0 0.0"/>
-      <geometry>
-        <box size="0.001 0.001 0.001"/>
-      </geometry>
-      <material name="black"/>
-    </visual>
-    <collision>
-      <geometry>
-        <box size="0.001 0.001 0.001"/>
-      </geometry>
-    </collision>
-    <xacro:sphere_inertial radius="0.02" mass="0.1" />
+    <xacro:sphere_inertial radius="0.02" mass="0.15" />
   </link>
   <link name="$(arg tf_prefix)imu">
@@ -276,5 +277,5 @@
     <child link="$(arg tf_prefix)axis_fl"/>
     <origin xyz="0.255 0.08 0.03" rpy="0.0 0.0 0.0"/>
-    <dynamics damping="0.1" friction="0.01"/>
+    <dynamics damping="0.1" friction="0.1"/>
   </joint>
   <joint name="$(arg tf_prefix)frontwheel_steering_right" type="revolute">
@@ -284,5 +285,5 @@
     <child link="$(arg tf_prefix)axis_fr"/>
     <origin xyz="0.255 -0.08 0.03" rpy="0.0 0.0 0.0" />
-    <dynamics damping="0.1" friction="0.01"/>
+    <dynamics damping="0.1" friction="0.1"/>
   </joint>
   <joint name="$(arg tf_prefix)frontwheel_left" type="continuous">
@@ -291,6 +292,6 @@
     <child link="$(arg tf_prefix)wheel_fl"/>
     <origin xyz="0 0 0" rpy="0.0 0.0 0.0"/>
-    <limit effort="100.0" velocity="100.0"/>
-    <dynamics damping="0.1" friction="0.01"/>
+    <limit effort="100.0" velocity="500.0"/>
+    <dynamics damping="0.1" friction="0.1"/>
   </joint>
   <joint name="$(arg tf_prefix)frontwheel_right" type="continuous">
@@ -299,6 +300,6 @@
     <child link="$(arg tf_prefix)wheel_fr"/>
     <origin xyz="0 0 0" rpy="0.0 0.0 0.0"/>
-    <limit effort="100.0" velocity="100.0"/>
-    <dynamics damping="0.1" friction="0.01"/>
+    <limit effort="100.0" velocity="500.0"/>
+    <dynamics damping="0.1" friction="0.1"/>
   </joint>
    <joint name="$(arg tf_prefix)rearwheel_left" type="continuous">
@@ -307,6 +308,6 @@
     <child link="$(arg tf_prefix)wheel_bl"/>
     <origin xyz="0 0.085 0.03" rpy="0.0 0.0 0.0"/>
-    <limit effort="100.0" velocity="100.0"/>
-     <dynamics damping="0.1" friction="0.01"/>
+    <limit effort="100.0" velocity="500.0"/>
+     <dynamics damping="0.1" friction="0.1"/>
    </joint>
   <joint name="$(arg tf_prefix)rearwheel_right" type="continuous">
@@ -315,6 +316,6 @@
     <child link="$(arg tf_prefix)wheel_br"/>
     <origin xyz="0 -0.085 0.03" rpy="0.0 0.0 0.0" />
-    <limit effort="100.0" velocity="100.0"/>
-    <dynamics damping="0.1" friction="0.01"/>
+    <limit effort="100.0" velocity="500.0"/>
+    <dynamics damping="0.1" friction="0.1"/>
   </joint>
   <joint name="$(arg tf_prefix)board_support_l" type="fixed">
