Commit message: Reformat xacro car file

File: catkin_ws/src/car_description/urdf/car.xacro (robot description, xacro)
@@ -1,332 +1,332 @@
 <?xml version="1.0"?>
 <robot name="$(arg car_name)" xmlns:xacro="http://www.ros.org/wiki/xacro">
-  <xacro:include filename="$(find car_description)/urdf/_d435.urdf.xacro"/>
-  <xacro:include filename="$(find car_description)/urdf/rplidar_a2.xacro"/>
-  <xacro:include filename="$(find car_description)/urdf/common.xacro"/>
-  <xacro:arg name="tf_prefix" default=""/>
-  <xacro:arg name="agent_prefix" default=""/>
-  <material name="black">
-    <color rgba="0.1 0.1 0.1 1"/>
-  </material>
-  <material name="plastic">
-    <color rgba="1 1 1 0.25"/>
-  </material>
-  <material name="imu">
-    <color rgba="0.2 0.5 0.1 1"/>
-  </material>
-  <material name="grey">
-    <color rgba="0.75 0.75 0.75 1"/>
-  </material>
-  <material name="white">
-    <color rgba="0.95 0.95 0.95 1"/>
-  </material>
-  <link name="$(arg tf_prefix)base_link">
-    <visual>
-      <origin rpy="0.0 0 0" xyz="0.135 0 0.01"/>
-      <geometry>
-        <mesh filename="file://$(find car_description)/meshes/chasi.dae"/>
-      </geometry>
-      <material name="black"/>
-    </visual>
-    <collision>
-      <origin rpy="0.0 0 0" xyz="0.135 0 0.01"/>
-      <geometry>
-        <mesh filename="file://$(find car_description)/meshes/chasi.dae"/>
-      </geometry>
-    </collision>
-    <xacro:box_inertial_with_origin mass="30.0" x="0.2" y="0.1" z="0.05">
-      <origin rpy="0.0 0 0" xyz="0.115 0 0.0" />
-    </xacro:box_inertial_with_origin>
-  </link>
-  <link name="$(arg tf_prefix)board">
-    <visual>
-      <origin rpy="0.0 0 0" xyz="0.115 0 0"/>
-      <geometry>
-        <mesh filename="file://$(find car_description)/meshes/board.dae"/>
-      </geometry>
-      <material name="plastic"/>
-    </visual>
-    <collision>
-      <origin rpy="0.0 0 0" xyz="0.115 0 0"/>
-      <geometry>
-        <mesh filename="file://$(find car_description)/meshes/board.dae"/>
-      </geometry>
-    </collision>
-    <xacro:box_inertial_with_origin x="0.3" y="0.1" z="0.1" mass="0.3" >
-      <origin xyz="0 0 0" rpy="0 0 0" />
-    </xacro:box_inertial_with_origin>
-  </link>
-  <link name="$(arg tf_prefix)camera_board">
-    <visual>
-      <origin rpy="0.0 0 0" xyz="0 0 0"/>
-      <geometry>
-        <mesh filename="file://$(find car_description)/meshes/camera_board.dae"/>
-      </geometry>
-      <material name="plastic"/>
-    </visual>
-    <collision>
-      <origin rpy="0.0 0 0" xyz="0 0 0"/>
-      <geometry>
-        <mesh filename="file://$(find car_description)/meshes/camera_board.dae"/>
-      </geometry>
-    </collision>
-    <inertial>
-      <origin rpy="0.0 0 0" xyz="0 0 0"/>
-      <mass value="0.1"/>
-      <inertia ixx="0.00014165" ixy="0.0" ixz="0.0" iyy="0.00006758" iyz="0.0" izz="0.00020865"/>
-    </inertial>
-  </link>
-  <xacro:macro name="wheel" params="name">
-    <link name="${name}">
-      <visual>
-        <origin rpy="0.0 0.0 0.0" xyz="0.0 0.0 0.0"/>
-        <geometry>
-          <mesh filename="file://$(find car_description)/meshes/wheel.dae"/>
-        </geometry>
-        <material name="black"/>
-      </visual>
-      <collision>
-        <origin rpy="0 1.5707 1.5707" xyz="0 0 0"/>
-        <geometry>
-          <cylinder length="0.025" radius="0.0325" />
-        </geometry>
-      </collision>
-      <xacro:cylinder_inertial_with_origin radius="0.025" length="0.0325" mass="0.1" >
-        <origin xyz="0 0 0" rpy="0 1.5707 1.5707" />
-      </xacro:cylinder_inertial_with_origin>
-    </link>
-    <gazebo reference="${name}">
-      <mu1>0.9</mu1>
-      <mu2>0.9</mu2>
-      <kp>1000000.0</kp> <!--contact stiffness-->
-      <kd>1.0</kd> <!--damping-->
-      <minDepth>0.001</minDepth>
-    </gazebo>
-  </xacro:macro>
-  <xacro:wheel name="$(arg tf_prefix)wheel_fr"/>
-  <xacro:wheel name="$(arg tf_prefix)wheel_fl"/>
-  <xacro:wheel name="$(arg tf_prefix)wheel_br"/>
-  <xacro:wheel name="$(arg tf_prefix)wheel_bl"/>
-  <link name="$(arg tf_prefix)axis_fl">
-    <visual>
-      <origin rpy="0.0 0.0 0.0" xyz="0.0 0.0 0.0"/>
-      <geometry>
-        <box size="0.001 0.001 0.001"/>
-      </geometry>
-      <material name="black"/>
-    </visual>
-    <collision>
-      <geometry>
-        <box size="0 0 0"/>
-      </geometry>
-    </collision>
-    <xacro:sphere_inertial radius="0.02" mass="0.15" />
-  </link>
-  <link name="$(arg tf_prefix)axis_fr">
-    <visual>
-      <origin rpy="0.0 0.0 0.0" xyz="0.0 0.0 0.0"/>
-      <geometry>
-        <box size="0 0 0"/>
-      </geometry>
-      <material name="black"/>
-    </visual>
-    <collision>
-      <geometry>
-        <box size="0.001 0.001 0.001"/>
-      </geometry>
-    </collision>
-    <xacro:sphere_inertial radius="0.02" mass="0.15" />
-  </link>
-  <link name="$(arg tf_prefix)imu">
-    <visual>
-      <geometry>
-        <box size="0.066 0.064 0.01"/>
-      </geometry>
-      <origin rpy="0 0 0" xyz="0 0 0"/>
-      <material name="imu"/>
-    </visual>
-    <collision>
-      <geometry>
-        <box size="0.066 0.064 0.01"/>
-      </geometry>
-    </collision>
-    <inertial>
-      <mass value="0.2"/>
-      <inertia ixx="0.00006993" ixy="0.0" ixz="0.0" iyy="0.00007427" iyz="0.0" izz="0.00014087"/>
-    </inertial>
-  </link>
-  <link name="$(arg tf_prefix)marker">
-    <visual>
-      <geometry>
-        <mesh filename="file://$(find car_description)/meshes/marker.dae"/>
-      </geometry>
-      <origin rpy="0 0 1.5708" xyz="0 0 0"/>
-    </visual>
-    <collision>
-      <geometry>
-        <box size="0.03 0.03 0.000001"/>
-      </geometry>
-    </collision>
-    <inertial>
-      <mass value="0.001"/>
-      <inertia ixx="0.00000008" ixy="0.0" ixz="0.0" iyy="0.00000008" iyz="0.0" izz="0.00000015"/>
-    </inertial>
-  </link>
-  <link name="$(arg tf_prefix)support_l">
-    <visual>
-      <geometry>
-        <cylinder length="0.22" radius="0.004"/>
-      </geometry>
-      <origin rpy="0 0 0" xyz="0 0 0"/>
-      <material name="black"/>
-    </visual>
-    <collision>
-      <geometry>
-        <cylinder length="0.22" radius="0.004"/>
-      </geometry>
-    </collision>
-    <inertial>
-      <mass value="0.001"/>
-      <inertia ixx="0.00000404" ixy="0.0" ixz="0.0" iyy="0.00000404" iyz="0.0" izz="0.00000001"/>
-    </inertial>
-  </link>
-  <link name="$(arg tf_prefix)support_r">
-    <visual>
-      <geometry>
-        <cylinder length="0.22" radius="0.004"/>
-      </geometry>
-      <origin rpy="0 0 0" xyz="0 0 0"/>
-      <material name="black"/>
-    </visual>
-    <collision>
-      <geometry>
-        <cylinder length="0.22" radius="0.004"/>
-      </geometry>
-    </collision>
-    <inertial>
-      <mass value="0.001"/>
-      <inertia ixx="0.00000404" ixy="0.0" ixz="0.0" iyy="0.00000404" iyz="0.0" izz="0.00000001"/>
-    </inertial>
-  </link>
-  <!-- BNO055 -->
-  <link name="$(arg tf_prefix)bno055">
-  </link>
-  <link name="$(arg tf_prefix)nuc">
-    <visual>
-      <origin rpy="0 0 0" xyz="0 0 0.022"/>
-      <geometry>
-        <box size="0.11 0.11 0.04" />
-      </geometry>
-      <material name="black"/>
-    </visual>
-    <collision>
-      <origin rpy="0 0 0" xyz="0 0 0.022"/>
-      <geometry>
-        <box size="0.11 0.11 0.04" />
-      </geometry>
-    </collision>
-    <xacro:box_inertial_with_origin x="0.11" y="0.11" z="0.04" mass="0.7" >
-      <origin xyz="0 0 0.025" rpy="0 0 0" />
-    </xacro:box_inertial_with_origin>
-  </link>
-  <!-- front camera -->
-  <xacro:property name="front_camera_name" value="camera"/>
-  <xacro:sensor_d435 parent="$(arg tf_prefix)camera_board" sensor_name="$(arg tf_prefix)camera">
-    <origin xyz="0.03 0 0.025" rpy="0 0.2 0"/>
-  </xacro:sensor_d435>
-  <xacro:sensor_d435 parent="$(arg tf_prefix)camera_board" sensor_name="rear_camera">
-    <origin xyz="-0.02 0 0.025" rpy="0 0.2 3.141"/>
-  </xacro:sensor_d435>
-  <xacro:sensor_rplidar_a2 parent="$(arg tf_prefix)board" prefix="lidar" tf_prefix="$(arg tf_prefix)">
-    <origin xyz="0.14 0 0.0425" rpy="0 0 0"/>
-  </xacro:sensor_rplidar_a2>
-  <joint name="$(arg tf_prefix)joint_board_to_bno055" type="fixed">
-      <parent link="$(arg tf_prefix)board"/>
-      <child link="$(arg tf_prefix)bno055"/>
-      <origin xyz="0.235 0.0 0.023" rpy="0 0 1.5708"/>
-  </joint>
-  <joint name="$(arg tf_prefix)base_link_board" type="fixed">
-    <parent link="$(arg tf_prefix)base_link"/>
-    <child link="$(arg tf_prefix)board"/>
-    <origin xyz="0 0 0.07"/>
-  </joint>
-  <joint name="$(arg tf_prefix)board_cameraboard" type="fixed">
-    <parent link="$(arg tf_prefix)board"/>
-    <child link="$(arg tf_prefix)camera_board"/>
-    <origin xyz="-0.025 0 0.15"/>
-  </joint>
-  <joint name="$(arg tf_prefix)board_imu" type="fixed">
-    <parent link="$(arg tf_prefix)board"/>
-    <child link="$(arg tf_prefix)imu"/>
-    <origin xyz="0.07 -0.017 0"/>
-  </joint>
-  <joint name="$(arg tf_prefix)board_marker" type="fixed">
-    <parent link="$(arg tf_prefix)board"/>
-    <child link="$(arg tf_prefix)marker"/>
-    <origin xyz="0.30 0.0 0.0025"/>
-  </joint>
-  <joint name="$(arg tf_prefix)board_nuc" type="fixed">
-    <parent link="$(arg tf_prefix)board"/>
-    <child link="$(arg tf_prefix)nuc"/>
-    <origin xyz="0.16 0 0"/>
-  </joint>
-  <joint name="$(arg tf_prefix)frontwheel_steering_left" type="revolute">
-    <axis xyz="0 0 1"/>
-    <limit effort="0.001" lower="-0.60" upper="0.60" velocity="1.0"/>
-    <parent link="$(arg tf_prefix)base_link"/>
-    <child link="$(arg tf_prefix)axis_fl"/>
-    <origin xyz="0.255 0.08 0.03" rpy="0.0 0.0 0.0"/>
-    <dynamics damping="0.1" friction="0.1"/>
-  </joint>
-  <joint name="$(arg tf_prefix)frontwheel_steering_right" type="revolute">
-    <axis xyz="0 0 1"/>
-    <limit effort="0.001" lower="-0.60" upper="0.60" velocity="1.0"/>
-    <parent link="$(arg tf_prefix)base_link"/>
-    <child link="$(arg tf_prefix)axis_fr"/>
-    <origin xyz="0.255 -0.08 0.03" rpy="0.0 0.0 0.0" />
-    <dynamics damping="0.1" friction="0.1"/>
-  </joint>
-  <joint name="$(arg tf_prefix)frontwheel_left" type="continuous">
-    <axis xyz="0 1 0"/>
-    <parent link="$(arg tf_prefix)axis_fl"/>
-    <child link="$(arg tf_prefix)wheel_fl"/>
-    <origin xyz="0 0 0" rpy="0.0 0.0 0.0"/>
-    <limit effort="100.0" velocity="500.0"/>
-    <dynamics damping="0.1" friction="0.1"/>
-  </joint>
-  <joint name="$(arg tf_prefix)frontwheel_right" type="continuous">
-    <axis xyz="0 1 0"/>
-    <parent link="$(arg tf_prefix)axis_fr"/>
-    <child link="$(arg tf_prefix)wheel_fr"/>
-    <origin xyz="0 0 0" rpy="0.0 0.0 0.0"/>
-    <limit effort="100.0" velocity="500.0"/>
-    <dynamics damping="0.1" friction="0.1"/>
-  </joint>
-   <joint name="$(arg tf_prefix)rearwheel_left" type="continuous">
-    <axis xyz="0 1 0"/>
-    <parent link="$(arg tf_prefix)base_link"/>
-    <child link="$(arg tf_prefix)wheel_bl"/>
-    <origin xyz="0 0.085 0.03" rpy="0.0 0.0 0.0"/>
-    <limit effort="100.0" velocity="500.0"/>
-     <dynamics damping="0.1" friction="0.1"/>
-   </joint>
-  <joint name="$(arg tf_prefix)rearwheel_right" type="continuous">
-    <axis xyz="0 1 0"/>
-    <parent link="$(arg tf_prefix)base_link"/>
-    <child link="$(arg tf_prefix)wheel_br"/>
-    <origin xyz="0 -0.085 0.03" rpy="0.0 0.0 0.0" />
-    <limit effort="100.0" velocity="500.0"/>
-    <dynamics damping="0.1" friction="0.1"/>
-  </joint>
-  <joint name="$(arg tf_prefix)board_support_l" type="fixed">
-    <parent link="$(arg tf_prefix)board"/>
-    <child link="$(arg tf_prefix)support_l"/>
-    <origin xyz="-0.024000 0.053000 0.112000"/>
-  </joint>
-  <joint name="$(arg tf_prefix)board_support_r" type="fixed">
-    <parent link="$(arg tf_prefix)board"/>
-    <child link="$(arg tf_prefix)support_r"/>
-    <origin xyz="-0.024000 -0.053000 0.112000"/>
-  </joint>
+    <xacro:include filename="$(find car_description)/urdf/_d435.urdf.xacro"/>
+    <xacro:include filename="$(find car_description)/urdf/rplidar_a2.xacro"/>
+    <xacro:include filename="$(find car_description)/urdf/common.xacro"/>
+    <xacro:arg name="tf_prefix" default=""/>
+    <xacro:arg name="agent_prefix" default=""/>
+    <material name="black">
+        <color rgba="0.1 0.1 0.1 1"/>
+    </material>
+    <material name="plastic">
+        <color rgba="1 1 1 0.25"/>
+    </material>
+    <material name="imu">
+        <color rgba="0.2 0.5 0.1 1"/>
+    </material>
+    <material name="grey">
+        <color rgba="0.75 0.75 0.75 1"/>
+    </material>
+    <material name="white">
+        <color rgba="0.95 0.95 0.95 1"/>
+    </material>
+    <link name="$(arg tf_prefix)base_link">
+        <visual>
+            <origin rpy="0.0 0 0" xyz="0.135 0 0.01"/>
+            <geometry>
+                <mesh filename="file://$(find car_description)/meshes/chasi.dae"/>
+            </geometry>
+            <material name="black"/>
+        </visual>
+        <collision>
+            <origin rpy="0.0 0 0" xyz="0.135 0 0.01"/>
+            <geometry>
+                <mesh filename="file://$(find car_description)/meshes/chasi.dae"/>
+            </geometry>
+        </collision>
+        <xacro:box_inertial_with_origin mass="30.0" x="0.2" y="0.1" z="0.05">
+            <origin rpy="0.0 0 0" xyz="0.115 0 0.0"/>
+        </xacro:box_inertial_with_origin>
+    </link>
+    <link name="$(arg tf_prefix)board">
+        <visual>
+            <origin rpy="0.0 0 0" xyz="0.115 0 0"/>
+            <geometry>
+                <mesh filename="file://$(find car_description)/meshes/board.dae"/>
+            </geometry>
+            <material name="plastic"/>
+        </visual>
+        <collision>
+            <origin rpy="0.0 0 0" xyz="0.115 0 0"/>
+            <geometry>
+                <mesh filename="file://$(find car_description)/meshes/board.dae"/>
+            </geometry>
+        </collision>
+        <xacro:box_inertial_with_origin x="0.3" y="0.1" z="0.1" mass="0.3">
+            <origin xyz="0 0 0" rpy="0 0 0"/>
+        </xacro:box_inertial_with_origin>
+    </link>
+    <link name="$(arg tf_prefix)camera_board">
+        <visual>
+            <origin rpy="0.0 0 0" xyz="0 0 0"/>
+            <geometry>
+                <mesh filename="file://$(find car_description)/meshes/camera_board.dae"/>
+            </geometry>
+            <material name="plastic"/>
+        </visual>
+        <collision>
+            <origin rpy="0.0 0 0" xyz="0 0 0"/>
+            <geometry>
+                <mesh filename="file://$(find car_description)/meshes/camera_board.dae"/>
+            </geometry>
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