Commit message: Initial jazzy update

File: catkin_ws/src/car_description/urdf/car.xacro (robot description, xacro)
@@ -273,17 +273,17 @@
     <joint name="$(arg tf_prefix)frontwheel_steering_left" type="revolute">
         <axis xyz="0 0 1"/>
-        <limit effort="0.001" lower="-0.60" upper="0.60" velocity="1.0"/>
+        <limit effort="100.0" lower="-0.6" upper="0.6" velocity="1.0"/>
         <parent link="$(arg tf_prefix)base_link"/>
         <child link="$(arg tf_prefix)axis_fl"/>
         <origin xyz="0.255 0.08 0.03" rpy="0.0 0.0 0.0"/>
-        <dynamics damping="0.1" friction="0.1"/>
+        <dynamics damping="0.2" friction="0.1"/>
     </joint>
     <joint name="$(arg tf_prefix)frontwheel_steering_right" type="revolute">
         <axis xyz="0 0 1"/>
-        <limit effort="0.001" lower="-0.60" upper="0.60" velocity="1.0"/>
+        <limit effort="100.0" lower="-0.6" upper="0.6" velocity="1.0"/>
         <parent link="$(arg tf_prefix)base_link"/>
         <child link="$(arg tf_prefix)axis_fr"/>
         <origin xyz="0.255 -0.08 0.03" rpy="0.0 0.0 0.0"/>
-        <dynamics damping="0.1" friction="0.1"/>
+        <dynamics damping="0.2" friction="0.1"/>
     </joint>
     <joint name="$(arg tf_prefix)frontwheel_left" type="continuous">
@@ -292,6 +292,6 @@
         <child link="$(arg tf_prefix)wheel_fl"/>
         <origin xyz="0 0 0" rpy="0.0 0.0 0.0"/>
-        <limit effort="100.0" velocity="500.0"/>
-        <dynamics damping="0.1" friction="0.1"/>
+        <limit effort="1.0" velocity="100.0"/>
+        <dynamics damping="0.2" friction="0.1"/>
     </joint>
     <joint name="$(arg tf_prefix)frontwheel_right" type="continuous">
@@ -300,6 +300,6 @@
         <child link="$(arg tf_prefix)wheel_fr"/>
         <origin xyz="0 0 0" rpy="0.0 0.0 0.0"/>
-        <limit effort="100.0" velocity="500.0"/>
-        <dynamics damping="0.1" friction="0.1"/>
+        <limit effort="1.0" velocity="100.0"/>
+        <dynamics damping="0.2" friction="0.1"/>
     </joint>
     <joint name="$(arg tf_prefix)rearwheel_left" type="continuous">
@@ -308,6 +308,6 @@
         <child link="$(arg tf_prefix)wheel_bl"/>
         <origin xyz="0 0.085 0.03" rpy="0.0 0.0 0.0"/>
-        <limit effort="100.0" velocity="500.0"/>
-        <dynamics damping="0.1" friction="0.1"/>
+        <limit effort="1.0" velocity="100.0"/>
+        <dynamics damping="0.2" friction="0.1"/>
     </joint>
     <joint name="$(arg tf_prefix)rearwheel_right" type="continuous">
@@ -316,6 +316,6 @@
         <child link="$(arg tf_prefix)wheel_br"/>
         <origin xyz="0 -0.085 0.03" rpy="0.0 0.0 0.0"/>
-        <limit effort="100.0" velocity="500.0"/>
-        <dynamics damping="0.1" friction="0.1"/>
+        <limit effort="1.0" velocity="100.0"/>
+        <dynamics damping="0.2" friction="0.1"/>
     </joint>
     <joint name="$(arg tf_prefix)board_support_l" type="fixed">
@@ -331,5 +331,5 @@
     <ros2_control name="GazeboSystem" type="system">
         <hardware>
-            <plugin>gazebo_ros2_control/GazeboSystem</plugin>
+          <plugin>gz_ros2_control/GazeboSimSystem</plugin>
         </hardware>
         <joint name="$(arg tf_prefix)rearwheel_left">
@@ -354,18 +354,10 @@
         </joint>
         <joint name="$(arg tf_prefix)frontwheel_steering_left">
-            <command_interface name="position">
-                <param name="min">-0.60</param>
-                <param name="max">0.60</param>
-            </command_interface>
+            <command_interface name="position"/>
             <state_interface name="position"/>
-            <state_interface name="velocity"/>
         </joint>
         <joint name="$(arg tf_prefix)frontwheel_steering_right">
-            <command_interface name="position">
-                <param name="min">-0.60</param>
-                <param name="max">0.60</param>
-            </command_interface>
+            <command_interface name="position"/>
             <state_interface name="position"/>
-            <state_interface name="velocity"/>
         </joint>
     </ros2_control>
@@ -388,11 +380,12 @@
         <implicitSpringDamper>true</implicitSpringDamper>
     </gazebo>
+      <gazebo>
+        <!-- Joint state publisher -->
+        <plugin filename="gz_ros2_control-system" name="gz_ros2_control::GazeboSimROS2ControlPlugin">
+          <parameters>$(find sim_car_controller)/config/control.yaml</parameters>
+        </plugin>
+      </gazebo>
     <gazebo>
-        <plugin filename="libgazebo_ros2_control.so" name="gazebo_ros2_control">
-            <parameters>$(find sim_car_controller)/config/control.yaml</parameters>
-        </plugin>
-    </gazebo>
-    <gazebo>
-        <plugin name="model_car_ground_truth" filename="libgazebo_ros_p3d.so">
+        <!--<plugin name="model_car_ground_truth" filename="libgazebo_ros_p3d.so">
             <ros>
                 <namespace>p3d</namespace>
@@ -402,18 +395,12 @@
             <body_name>$(arg tf_prefix)base_link</body_name>
             <update_rate>30.0</update_rate>
-        </plugin>
+        </plugin>-->
     </gazebo>
     <gazebo reference="$(arg tf_prefix)imu">
         <sensor name="$(arg tf_prefix)imu" type="imu">
-            <plugin filename="libgazebo_ros_imu_sensor.so" name="imu_plugin">
-                <ros>
-                    <namespace>sensors</namespace>
-                    <remapping>~/out:=imu</remapping>
-                </ros>
-                <initial_orientation_as_reference>false</initial_orientation_as_reference>
-            </plugin>
-            <always_on>true</always_on>
+            <always_on>1</always_on>
             <update_rate>100</update_rate>
             <visualize>true</visualize>
+            <topic>/sensors/imu</topic>
         </sensor>
     </gazebo>
@@ -423,4 +410,5 @@
             <visualize>true</visualize>
             <update_rate>15.0</update_rate>
+            <frame_name>$(arg tf_prefix)camera_depth_optical_frame</frame_name>
             <camera>
                 <pose>0 0 0 0 0.20 0</pose>
@@ -442,18 +430,4 @@
                     <stddev>0.007</stddev>
                 </noise>
-            </camera>
-            <plugin name="depth" filename="libgazebo_ros_camera.so">
-                <ros>
-                    <namespace>/sensors</namespace>
-                    <remapping>camera/image_raw:=camera/infra1/image_rect_raw</remapping>
-                    <remapping>camera/camera_info:=camera/infra1/camera_info</remapping>
-                    <remapping>camera/depth/image_raw:=camera/depth/image_rect_raw</remapping>
-                    <remapping>camera/depth/camera_info:=camera/depth/camera_info</remapping>
-                    <remapping>camera/points:=camera/depth/points</remapping>
-                </ros>
-                <always_on>true</always_on>
-                <update_rate>15.0</update_rate>
-                <camera_name>camera</camera_name>
-                <frame_name>$(arg tf_prefix)camera_depth_optical_frame</frame_name>
                 <pointCloudCutoff>0.05</pointCloudCutoff>
                 <pointCloudCutoffMax>15.0</pointCloudCutoffMax>
@@ -463,10 +437,5 @@
                 <Cy>241.67051696777344</Cy>
                 <focal_length>383.795710</focal_length>
-                <noise>
-                    <type>gaussian</type>
-                    <mean>0.0</mean>
-                    <stddev>0.0</stddev>
-                </noise>
-            </plugin>
+            </camera>
         </sensor>
     </gazebo>
@@ -491,13 +460,4 @@
                     <stddev>0.01</stddev>
                 </noise>
-            </camera>
-            <plugin name="color" filename="libgazebo_ros_camera.so">
-                <ros>
-                    <namespace>/sensors/camera</namespace>
-                    <remapping>color/image_raw:=color/image_rect_color</remapping>
-                </ros>
-                <always_on>true</always_on>
-                <update_rate>15.0</update_rate>
-                <camera_name>color</camera_name>
                 <frame_name>$(arg tf_prefix)camera_color_optical_frame</frame_name>
                 <hack_baseline>0.0193</hack_baseline>
@@ -507,24 +467,42 @@
                 <distortionT1>0.0</distortionT1>
                 <distortionT2>0.0</distortionT2>
-            </plugin>
+                <camera_name>color</camera_name>
+            </camera>
+            <!--<plugin name="color" filename="libgazebo_ros_camera.so">
+                <ros>
+                    <namespace>/sensors/camera</namespace>
+                    <remapping>color/image_raw:=color/image_rect_color</remapping>
+                </ros>
+                <always_on>true</always_on>
+                <update_rate>15.0</update_rate>
+            </plugin>-->
         </sensor>
     </gazebo>
     <gazebo reference="$(arg tf_prefix)laser">
-        <sensor type="ray" name="rp_lidar_sensor">
-            <pose>0 0 0 0 0 0</pose>
-            <visualize>false</visualize>
+        <sensor type="gpu_lidar" name="rp_lidar_sensor">
+            <pose relative_to='$(arg tf_prefix)laser'>0 0 0 0 0 0</pose>
+            <visualize>true</visualize>
             <update_rate>10</update_rate>
+            <topic>/sensors/rplidar/scan</topic>
+            <always_on>1</always_on>
             <ray>
                 <scan>
                     <horizontal>
                         <samples>360</samples>
+                        <resolution>1</resolution>
                         <min_angle>-3.14159</min_angle>
                         <max_angle>3.14159</max_angle>
                     </horizontal>
+                    <vertical>
+                        <samples>1</samples>
+                        <resolution>0.01</resolution>
+                        <min_angle>0</min_angle>
+                        <max_angle>0</max_angle>
+                    </vertical>
                 </scan>
                 <range>
                     <min>0.15</min>
                     <max>8.0</max>
-                    <resolution>0.05</resolution>
+                    <resolution>0.01</resolution>
                 </range>
                 <noise>
@@ -534,11 +512,4 @@
                 </noise>
             </ray>
-            <plugin name="rplidar" filename="libgazebo_ros_ray_sensor.so">
-                <ros>
-                    <remapping>~/out:=sensors/rplidar/scan</remapping>
-                </ros>
-                <output_type>sensor_msgs/LaserScan</output_type>
-                <frame_name>$(arg tf_prefix)laser</frame_name>
-            </plugin>
         </sensor>
     </gazebo>

Commit message: Fix camera frame and position

File: catkin_ws/src/car_description/urdf/car.xacro (robot description, xacro)
@@ -233,8 +233,8 @@
     <xacro:property name="front_camera_name" value="camera"/>
     <xacro:sensor_d435 parent="$(arg tf_prefix)camera_board" sensor_name="$(arg tf_prefix)camera">
-        <origin xyz="0.03 0 0.025" rpy="0 0.2 0"/>
+        <origin xyz="0.03 0 0.025" rpy="0 0.25 0"/>
     </xacro:sensor_d435>
     <xacro:sensor_d435 parent="$(arg tf_prefix)camera_board" sensor_name="rear_camera">
-        <origin xyz="-0.02 0 0.025" rpy="0 0.2 3.141"/>
+        <origin xyz="-0.02 0 0.025" rpy="0 0.25 3.141"/>
     </xacro:sensor_d435>
     <xacro:sensor_rplidar_a2 parent="$(arg tf_prefix)board" prefix="lidar" tf_prefix="$(arg tf_prefix)">
@@ -410,8 +410,8 @@
             <visualize>true</visualize>
             <update_rate>15.0</update_rate>
-            <!--<frame_name>$(arg tf_prefix)camera_depth_optical_frame</frame_name>-->
             <topic>/sensors/camera/depth/image_rect_raw</topic>
+            <gz_frame_id>$(arg tf_prefix)camera_depth_optical_frame</gz_frame_id>
             <camera>
-                <pose>0 0 0 0 0.20 0</pose>
+                <pose>0 0 0 0 0.25 0</pose>
                 <horizontal_fov>1.3900031938640904</horizontal_fov>
                 <image>
@@ -436,6 +436,7 @@
             <update_rate>15.0</update_rate>
             <topic>/sensors/camera/color/image_raw</topic>
+            <gz_frame_id>$(arg tf_prefix)camera_color_optical_frame</gz_frame_id>
             <camera>
-                <pose>0 0 0.02 0 0.20 0</pose>
+                <pose>0 0 0.02 0 0.25 0</pose>
                 <horizontal_fov>0.95417536656506718</horizontal_fov>
                 <image>
@@ -453,6 +454,5 @@
                     <stddev>0.01</stddev>
                 </noise>
-                <!--<frame_name>$(arg tf_prefix)camera_color_optical_frame</frame_name>
-                <hack_baseline>0.0193</hack_baseline>
+                <!--<hack_baseline>0.0193</hack_baseline>
                 <distortionK1>0.0</distortionK1>
                 <distortionK2>0.0</distortionK2>
@@ -462,12 +462,4 @@
                 <camera_name>color</camera_name>-->
             </camera>
-            <!--<plugin name="color" filename="libgazebo_ros_camera.so">
-                <ros>
-                    <namespace>/sensors/camera</namespace>
-                    <remapping>color/image_raw:=color/image_rect_color</remapping>
-                </ros>
-                <always_on>true</always_on>
-                <update_rate>15.0</update_rate>
-            </plugin>-->
         </sensor>
     </gazebo>

Commit message: Fix meshes

File: catkin_ws/src/car_description/urdf/car.xacro (robot description, xacro)
@@ -27,5 +27,4 @@
                 <mesh filename="file://$(find car_description)/meshes/chasi.dae"/>
             </geometry>
-            <material name="black"/>
         </visual>
         <collision>
@@ -84,5 +83,4 @@
                     <mesh filename="file://$(find car_description)/meshes/wheel.dae"/>
                 </geometry>
-                <material name="black"/>
             </visual>
             <collision>

Commit message: Increase wheel effort limits

File: catkin_ws/src/car_description/urdf/car.xacro (robot description, xacro)
@@ -290,6 +290,6 @@
         <child link="$(arg tf_prefix)wheel_fl"/>
         <origin xyz="0 0 0" rpy="0.0 0.0 0.0"/>
-        <limit effort="1.0" velocity="100.0"/>
-        <dynamics damping="0.2" friction="0.1"/>
+        <limit effort="100.0" velocity="100.0"/>
+        <dynamics damping="0.1" friction="0.1"/>
     </joint>
     <joint name="$(arg tf_prefix)frontwheel_right" type="continuous">
@@ -298,6 +298,6 @@
         <child link="$(arg tf_prefix)wheel_fr"/>
         <origin xyz="0 0 0" rpy="0.0 0.0 0.0"/>
-        <limit effort="1.0" velocity="100.0"/>
-        <dynamics damping="0.2" friction="0.1"/>
+        <limit effort="100.0" velocity="100.0"/>
+        <dynamics damping="0.1" friction="0.1"/>
     </joint>
     <joint name="$(arg tf_prefix)rearwheel_left" type="continuous">
@@ -306,6 +306,6 @@
         <child link="$(arg tf_prefix)wheel_bl"/>
         <origin xyz="0 0.085 0.03" rpy="0.0 0.0 0.0"/>
-        <limit effort="1.0" velocity="100.0"/>
-        <dynamics damping="0.2" friction="0.1"/>
+        <limit effort="100.0" velocity="100.0"/>
+        <dynamics damping="0.1" friction="0.1"/>
     </joint>
     <joint name="$(arg tf_prefix)rearwheel_right" type="continuous">
@@ -314,6 +314,6 @@
         <child link="$(arg tf_prefix)wheel_br"/>
         <origin xyz="0 -0.085 0.03" rpy="0.0 0.0 0.0"/>
-        <limit effort="1.0" velocity="100.0"/>
-        <dynamics damping="0.2" friction="0.1"/>
+        <limit effort="100.0" velocity="100.0"/>
+        <dynamics damping="0.1" friction="0.1"/>
     </joint>
     <joint name="$(arg tf_prefix)board_support_l" type="fixed">

Commit message: Model wheel collision as sphere to improve contact with ground

File: catkin_ws/src/car_description/urdf/car.xacro (robot description, xacro)
@@ -87,5 +87,5 @@
                 <origin rpy="0 1.5707 1.5707" xyz="0 0 0"/>
                 <geometry>
-                    <cylinder length="0.025" radius="0.0325"/>
+                    <sphere radius="0.0325"/>
                 </geometry>
             </collision>

Commit message: Fix front wheel speeds

File: catkin_ws/src/car_description/urdf/car.xacro (robot description, xacro)
@@ -87,5 +87,5 @@
                 <origin rpy="0 1.5707 1.5707" xyz="0 0 0"/>
                 <geometry>
-                    <sphere radius="0.0325"/>
+                    <cylinder length="0.025" radius="0.0325"/>
                 </geometry>
             </collision>
